File: planewatcher/kicad/Log_Detector.kicad_sch (KiCad schematic)
At the start: 13 parts, among them U18 ADL5513

Commit message: work on board layout
Parts:
- added C70: 10nF, Capacitor_SMD:C_0402_1005Metric, symbol Device:C
- renumbered C100 to C40, C101 to C41, C98 to C42, C99 to C43, C102 to C44, C103 to C45, R53 to R25, R54 to R26, R55 to R27, TP30 to TP13, TP29 to TP14, U18 to U9
Connections:
- net GND: now also C70.2
- net at R26.2, RV1.2, TP14.1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: now also C70.1

Commit message: add jumpers for testing different power rails & additional test point
Changed lines of the file:
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@@
 		)
 	)
-	(text_box "Voltage divider to set TADJ pin for optimum performance depening on frequency.\n\nFor first prototype, a trimmer is included to allow precise tuning.\nTrimmer at minimum: 0.8018V\nTrimmer at maximum: 0.8713V\n\nThis allows tuning between 900MHz & 1.9MHz from table 4 in datasheet (see inset)."
+	(text_box "Voltage divider to set TADJ pin for optimum performance depening on frequency.\n\nFor first prototype, a trimmer is included to allow precise tuning.\nTrimmer at minimum: 0.8018V\nTrimmer at maximum: 0.8713V\n\nThis allows tuning between 900MHz & 1.9MHz from table 4 in datasheet (see inset).\n\nReplace with simple voltage divider when optimum TADJ voltage is known."
 		(exclude_from_sim no)
 		(at 135.89 87.63 0)
-		(size 35.56 71.12)
+		(size 35.56 77.47)
 		(margins 0.9525 0.9525 0.9525 0.9525)
 		(stroke
 			(width 0)
 			(type solid)
+			(color 255 0 0 1)
 		)
 		(fill
@@
 			(font
 				(size 1.27 1.27)
+				(color 255 0 0 1)
 			)
 			(justify left bottom)

Commit message: address & fix ERC errors/warnings
Parts:
- RV1: Notes (none) -> For prototype: Voltage divider to set TADJ pin for optimum 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
Connections:
- net at RV1.1: now also C70.1, R26.2, RV1.2, TP14.1, U9.9 (TADJ)
Changed lines of the file:
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@@
+	)
+	(junction
+		(at 160.02 109.22)
+		(diameter 0)
+		(color 0 0 0 0)
 	)
 	(junction
@@
 	(wire
 		(pts
-			(xy 160.02 113.03) (xy 160.02 106.68)
+			(xy 160.02 113.03) (xy 160.02 109.22)
 		)
 		(stroke
@@
 	(wire
 		(pts
+			(xy 160.02 109.22) (xy 160.02 106.68)
+		)
+		(stroke
+			(width 0)
+			(type default)
+		)
+	)
+	(wire
+		(pts
 			(xy 40.64 68.58) (xy 44.45 68.58)
 		)
@@
 		(pts
 			(xy 40.64 76.2) (xy 66.04 76.2)
+		)
+		(stroke
+			(width 0)
+			(type default)
+		)
+	)
+	(wire
+		(pts
+			(xy 153.67 109.22) (xy 160.02 109.22)
 		)
 		(stroke
@@
 			)
 		)
+		(property "Notes" "For prototype: Voltage divider to set TADJ pin for optimum performance depening on frequency. "
+			(at 153.67 113.03 0)
+			(hide yes)
+			(show_name no)
+			(do_not_autoplace no)
+			(effects
+				(font
+					(size 1.27 1.27)
+				)
+			)
+		)
 		(pin "3"
 		)
@@
 		(pin "2"
 		)
-		(pin "5"
-		)
-		(pin "6"
-		)
-		(pin "7"
-		)
-		(pin "16"
-		)
-		(pin "13"
-		)
-		(pin "15"
-		)
-		(pin "8"
-		)
 		(instances

Commit message: fix all ERC & DRCC errors & warnings
Parts:
- added R41, R42: DNP, Resistor_SMD:R_0402_1005Metric, symbol Device:R
- added R43: 0Ω, Resistor_SMD:R_0402_1005Metric, symbol Device:R
Connections:
- net GND: now also R41.1, R42.1
- net RF_IN: now also R41.2, R43.1; no longer C42.1, R25.1
- net VPOS: no longer R26.1
- new net: C42.1, R25.1, R42.2, R43.2
- new net +5V: R26.1
Other:
- moved on the sheet: C40, C41, C42, C43, C44, C45, C70, R25, R26, R27, RV1, TP13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

Commit message: updates before fab
Parts:
- C40, C44: Purpose (none) -> Local high-frequency VPOS decoupling for the ADL5513 log de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; Suggested Part (none) -> Murata GRM155R71H104KE14D
- C41, C45: Purpose (none) -> ADL5513 VPOS high-frequency decoupling capacitor placed clo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; Suggested Part (none) -> Murata GRM1555C1H101JA01D
- C42, C43: Purpose (none) -> AC-couples ADL5513 RF input pins while preserving the broad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; Suggested Part (none) -> Murata GRM155R71H473KE14D
- C70: Purpose (none) -> ADL5513 VOUT/VSET measurement-mode support capacitor in the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; Suggested Part (none) -> Murata GRM155R71H103KA88D
- R25: Purpose 52.3Ω, ±1%, 0402, RF input shunt termination, broadband 50Ω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 -> ADL5513 RF input shunt termination for broadband 50Ω matchi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; Suggested Part (none) -> Panasonic ERA-2AEB52R3X
- R26: Purpose Voltage divider for ADL5513 TADJ -> Upper resistor in the ADL5513 TADJ divider for 1090MHz dete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; Suggested Part (none) -> ${RTADJ_VPOS_Suggested_Part}
- R27: Purpose Voltage divider for ADL5513 TADJ -> Lower resistor in the ADL5513 TADJ divider for 1090MHz dete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; Suggested Part (none) -> ${RTADJ_GND_Suggested_Part}
- R41, R42: Purpose (none) -> Optional shunt leg for configurable RF input attenuation ah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; Suggested Part (none) -> DNP by default; fit Vishay CRCW0402 value selected from att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
- R43: Purpose (none) -> Zero-ohm link tying ADL5513 VOUT to VSET for measurement mo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; Suggested Part (none) -> Yageo RC0402JR-070RL
- RV1: Notes For prototype: Voltage divider to set TADJ pin for optimum performance depening on frequency. -> For prototype: Voltage divider to set TADJ pin for optimum performance depending on frequency.; Purpose (none) -> Allows prototype adjustment of the ADL5513 TADJ calibration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; Suggested Part (none) -> Bourns 3224W-1-102E
- TP13: Purpose (none) -> Provides oscilloscope/DMM probe access to VLOG_OUT.; Suggested Part (none) -> No fitted part (PCB pad only); now left out of the parts list
- TP14: Purpose (none) -> Provides oscilloscope/DMM probe access to TADJ.; Suggested Part (none) -> No fitted part (PCB pad only); now left out of the parts list
- U9: Purpose (none) -> Converts 1090MHz RF amplitude into a logarithmic video/RSSI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; Suggested Part (none) -> Analog Devices ADL5513ACPZ-R7

Commit message: rationalise power to single 3V3 rail fed from FPGA VCC
Connections:
- net +5V is gone; now on net VPOS: R26.1
Changed lines of the file:
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@@
 		)
 	)
-	(text_box "Voltage divider to set TADJ pin for optimum performance depending on frequency.\n\nFor first prototype, a trimmer is included to allow precise tuning.\nTrimmer at minimum: 0.8018V\nTrimmer at maximum: 0.8713V\n\nThis allows tuning between 900MHz & 1.9GHz from table 4 in datasheet (see inset).\n\nReplace with simple voltage divider when optimum TADJ voltage is known."
+	(text_box "Voltage divider to set TADJ pin for optimum performance depending on frequency.\n\nFor first prototype, a trimmer is included to allow precise tuning from a 3.32V VPOS rail.\nTrimmer at minimum: 0.8017V\nTrimmer at maximum: 0.8713V\n\nThis allows tuning between 900MHz & 1.9GHz from table 4 in datasheet (see inset).\n\nReplace with simple voltage divider when optimum TADJ voltage is known."
 		(exclude_from_sim no)
 		(at 196.85 81.28 0)
-		(size 35.56 77.47)
+		(size 35.56 81.28)
 		(margins 0.9525 0.9525 0.9525 0.9525)
 		(stroke
@@
 		)
 	)
-	(hierarchical_label "+5V"
-		(shape input)
-		(at 220.98 90.17 90)
+	(hierarchical_label "VLOG_OUT"
+		(shape output)
+		(at 200.66 36.83 0)
 		(effects
 			(font
@@
 		)
 	)
-	(hierarchical_label "VLOG_OUT"
-		(shape output)
-		(at 200.66 36.83 0)
+	(hierarchical_label "VPOS"
+		(shape input)
+		(at 220.98 90.17 90)
 		(effects
 			(font
