File: planewatcher/kicad/LNA_Stage.kicad_sch (KiCad schematic)
At the start: 8 parts, among them U7 TQP3M9036

Commit message: Add persistent PCBWay BOM fields to KiCad schematic
Parts:
- C28: MPN (none) -> GRM155R61C105KA12D; Manufacturer (none) -> Murata; Package (none) -> 0402
- C29: MPN (none) -> GRM155R71H104KE14D; Manufacturer (none) -> Murata; Package (none) -> 0402
- C30: MPN (none) -> GRM1555C1H102JA01D; Manufacturer (none) -> Murata; Package (none) -> 0402
- C31, C32, C33: MPN (none) -> GRM1555C1H101JA01D; Manufacturer (none) -> Murata; Package (none) -> 0402
- L7: MPN (none) -> 0603CS-68NXJLU; Manufacturer (none) -> Coilcraft; Package (none) -> 0603
- U7: MPN (none) -> TQP3M9036; Manufacturer (none) -> Qorvo; Package (none) -> QFN-16

Commit message: move power supply and add GPS module
Other:
- title: Plane Watcher: LNA Stage -> Plane Watcher
Changed lines of the file:
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@@
 	(paper "A4")
 	(title_block
-		(title "Plane Watcher: LNA Stage")
-		(date "2026-05-16")
-		(rev "prototype 1.1")
+		(title "Plane Watcher")
+		(date "2026-05-18")
+		(rev "prototype 1.2")
 		(company "plane.watch")
 	)

Commit message: review & consolidate all capacitors
Parts:
- C28: MPN GRM155R61C105KA12D -> GRM155Z71A105KE01D; Manufacturer Murata -> Murata Electronics; Package 0402 -> 0402 (1005 Metric); Suggested Part Murata GRM155R61C105KA12D -> (none)
- C29: MPN GRM155R71H104KE14D -> GCM155R71A104KA55D; Manufacturer Murata -> Murata Electronics; Package 0402 -> 0402 (1005 Metric); Suggested Part Murata GRM155R71H104KE14D -> (none)
- C30: MPN GRM1555C1H102JA01D -> GRM1555C1H102FA01D; Manufacturer Murata -> Murata Electronics; Package 0402 -> 0402 (1005 Metric); Suggested Part Murata GRM1555C1H102JA01D -> (none)
- C31, C32, C33: MPN GRM1555C1H101JA01D -> GCM1555C1H101FA16D; Manufacturer Murata -> Murata Electronics; Package 0402 -> 0402 (1005 Metric); Suggested Part Murata GRM1555C1H101JA01D -> (none)
- L7: Suggested Part Coilcraft 0603CS-68NXJLU -> (none)
- U7: Suggested Part Qorvo TQP3M9036 -> (none)
Changed lines of the file:
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@@
 			)
 		)
-		(property "Datasheet" ""
+		(property "Datasheet" "https://search.murata.co.jp/Ceramy/image/img/A01X/G101/ENG/GRM155Z71A105KE01-01.pdf"
 			(at 167.64 45.72 0)
 			(hide yes)
@@
 			)
 		)
-		(property "Description" "1µF, X5R, ±10%, 16V, 0402 MLCC"
+		(property "Description" "1 µF ±10% 10V Ceramic Capacitor X7R 0402 (1005 Metric)"
 			(at 167.64 45.72 0)
 			(hide yes)
@@
 			)
 		)
-		(property "Package" "0402"
+		(property "Package" "0402 (1005 Metric)"
 			(at 167.64 45.72 0)
 			(hide yes)
@@
 			)
 		)
-		(property "MPN" "GRM155R61C105KA12D"
+		(property "MPN" "GRM155Z71A105KE01D"
 			(at 167.64 45.72 0)
 			(hide yes)
@@
 			)
 		)
-		(property "Manufacturer" "Murata"
-			(at 167.64 45.72 0)
-			(hide yes)
-			(show_name no)
-			(do_not_autoplace no)
-			(effects
-				(font
-					(size 1.27 1.27)
-				)
-			)
-		)
-		(property "Suggested Part" "Murata GRM155R61C105KA12D"
+		(property "Manufacturer" "Murata Electronics"
 			(at 167.64 45.72 0)
 			(hide yes)
@@
 		)
 		(property "Notes" ""
+			(at 167.64 45.72 90)
+			(hide yes)
+			(show_name no)
+			(do_not_autoplace no)
+			(effects
+				(font
+					(size 1.27 1.27)
+				)
+			)
+		)
+		(property "Mount_Type" ""
 			(at 167.64 45.72 90)
 			(hide yes)
@@
 			)
 		)
-		(property "Datasheet" ""
+		(property "Datasheet" "https://search.murata.co.jp/Ceramy/image/img/A01X/G101/ENG/GCM1555C1HR50BA16-01A.pdf"
 			(at 120.65 104.14 0)
 			(hide yes)
@@
 			)
 		)
-		(property "Description" "100pF, C0G/NP0, ±5%, 50V, 0402 MLCC"
+		(property "Description" "100 pF ±1% 50V Ceramic Capacitor C0G, NP0 0402 (1005 Metric)"
 			(at 120.65 104.14 0)
 			(hide yes)
@@
 			)
 		)
-		(property "Package" "0402"
+		(property "Package" "0402 (1005 Metric)"
 			(at 120.65 104.14 0)
 			(hide yes)
@@
 			)
 		)
-		(property "MPN" "GRM1555C1H101JA01D"
+		(property "MPN" "GCM1555C1H101FA16D"
 			(at 120.65 104.14 0)
 			(hide yes)
@@
 			)
 		)
-		(property "Manufacturer" "Murata"
-			(at 120.65 104.14 0)
-			(hide yes)
-			(show_name no)
-			(do_not_autoplace no)
-			(effects
-				(font
-					(size 1.27 1.27)
-				)
-			)
-		)
-		(property "Suggested Part" "Murata GRM1555C1H101JA01D"
+		(property "Manufacturer" "Murata Electronics"
 			(at 120.65 104.14 0)
 			(hide yes)
@@
 		)
 		(property "Notes" ""
+			(at 120.65 104.14 90)
+			(hide yes)
+			(show_name no)
+			(do_not_autoplace no)
+			(effects
+				(font
+					(size 1.27 1.27)
+				)
+			)
+		)
+		(property "Mount_Type" ""
 			(at 120.65 104.14 90)
 			(hide yes)
@@
 			)
 		)
-		(property "Datasheet" ""
+		(property "Datasheet" "https://search.murata.co.jp/Ceramy/image/img/A01X/G101/ENG/GCM1555C1HR50BA16-01A.pdf"
 			(at 167.64 104.14 0)
 			(hide yes)
@@
 			)
 		)
-		(property "Description" "100pF, C0G/NP0, ±5%, 50V, 0402 MLCC"
+		(property "Description" "100 pF ±1% 50V Ceramic Capacitor C0G, NP0 0402 (1005 Metric)"
 			(at 167.64 104.14 0)
 			(hide yes)
@@
 			)
 		)
-		(property "Package" "0402"
+		(property "Package" "0402 (1005 Metric)"
 			(at 167.64 104.14 0)
 			(hide yes)
@@
 			)
 		)
-		(property "MPN" "GRM1555C1H101JA01D"
+		(property "MPN" "GCM1555C1H101FA16D"
 			(at 167.64 104.14 0)
 			(hide yes)
@@
 			)
 		)
-		(property "Manufacturer" "Murata"
-			(at 167.64 104.14 0)
-			(hide yes)
-			(show_name no)
-			(do_not_autoplace no)
-			(effects
-				(font
-					(size 1.27 1.27)
-				)
-			)
-		)
-		(property "Suggested Part" "Murata GRM1555C1H101JA01D"
+		(property "Manufacturer" "Murata Electronics"
 			(at 167.64 104.14 0)
 			(hide yes)
@@
 		)
 		(property "Notes" ""
+			(at 167.64 104.14 90)
+			(hide yes)
+			(show_name no)
+			(do_not_autoplace no)
+			(effects
+				(font
+					(size 1.27 1.27)
+				)
+			)
+		)
+		(property "Mount_Type" ""
 			(at 167.64 104.14 90)
 			(hide yes)
@@
 			)
 		)
-		(property "Datasheet" ""
+		(property "Datasheet" "https://search.murata.co.jp/Ceramy/image/img/A01X/G101/ENG/GCM155R71A104KA55-01.pdf"
 			(at 167.64 58.42 0)
 			(hide yes)
@@
 			)
 		)
-		(property "Description" "100nF, X7R, ±10%, 50V, 0402 MLCC"
+		(property "Description" "0.1 µF ±10% 10V Ceramic Capacitor X7R 0402 (1005 Metric)"
 			(at 167.64 58.42 0)
 			(hide yes)
@@
 			)
 		)
-		(property "Package" "0402"
+		(property "Package" "0402 (1005 Metric)"
 			(at 167.64 58.42 0)
 			(hide yes)
@@
 			)
 		)
-		(property "MPN" "GRM155R71H104KE14D"
+		(property "MPN" "GCM155R71A104KA55D"
 			(at 167.64 58.42 0)
 			(hide yes)
@@
 			)
 		)
-		(property "Manufacturer" "Murata"
-			(at 167.64 58.42 0)
-			(hide yes)
-			(show_name no)
-			(do_not_autoplace no)
-			(effects
-				(font
-					(size 1.27 1.27)
-				)
-			)
-		)
-		(property "Suggested Part" "Murata GRM155R71H104KE14D"
+		(property "Manufacturer" "Murata Electronics"
 			(at 167.64 58.42 0)
 			(hide yes)
@@
 		(property "Purpose" "Local high-frequency decoupling for the TQP3M9036 LNA supply."
 			(at 167.64 58.42 0)
+			(hide yes)
+			(show_name no)
+			(do_not_autoplace no)
+			(effects
+				(font
+					(size 1.27 1.27)
+				)
+			)
+		)
+		(property "Mount_Type" ""
+			(at 167.64 58.42 90)
 			(hide yes)
 			(show_name no)
@@
 			)
 		)
-		(property "Datasheet" ""
+		(property "Datasheet" "https://search.murata.co.jp/Ceramy/image/img/A01X/G101/ENG/GRM1555C1H102FA01-01.pdf"
 			(at 167.64 71.12 0)
 			(hide yes)
@@
 			)
 		)
-		(property "Description" "1nF, C0G/NP0, ±5%, 50V, 0402 MLCC"
+		(property "Description" "1000 pF ±1% 50V Ceramic Capacitor C0G, NP0 0402 (1005 Metric)"
 			(at 167.64 71.12 0)
 			(hide yes)
@@
 			)
 		)
-		(property "Package" "0402"
+		(property "Package" "0402 (1005 Metric)"
 			(at 167.64 71.12 0)
 			(hide yes)
@@
 			)
 		)
-		(property "MPN" "GRM1555C1H102JA01D"
+		(property "MPN" "GRM1555C1H102FA01D"
 			(at 167.64 71.12 0)
 			(hide yes)
@@
 			)
 		)
-		(property "Manufacturer" "Murata"
-			(at 167.64 71.12 0)
-			(hide yes)
-			(show_name no)
-			(do_not_autoplace no)
-			(effects
-				(font
-					(size 1.27 1.27)
-				)
-			)
-		)
-		(property "Suggested Part" "Murata GRM1555C1H102JA01D"
+		(property "Manufacturer" "Murata Electronics"
 			(at 167.64 71.12 0)
 			(hide yes)
@@
 		(property "Purpose" "RF supply bypass/matching capacitor for the 1090MHz LNA stage."
 			(at 167.64 71.12 0)
+			(hide yes)
+			(show_name no)
+			(do_not_autoplace no)
+			(effects
+				(font
+					(size 1.27 1.27)
+				)
+			)
+		)
+		(property "Mount_Type" ""
+			(at 167.64 71.12 90)
 			(hide yes)
 			(show_name no)
@@
 			)
 		)
-		(property "Suggested Part" "Qorvo TQP3M9036"
-			(at 138.43 100.33 0)
-			(hide yes)
-			(show_name no)
-			(do_not_autoplace no)
-			(effects
-				(font
-					(size 1.27 1.27)
-				)
-			)
-		)
 		(property "Purpose" "Provides gain for the 1090MHz RF signal before filtering and detection."
 			(at 138.43 100.33 0)
@@
 		)
 		(property "Notes" ""
+			(at 138.43 100.33 0)
+			(hide yes)
+			(show_name no)
+			(do_not_autoplace no)
+			(effects
+				(font
+					(size 1.27 1.27)
+				)
+			)
+		)
+		(property "Mount_Type" ""
 			(at 138.43 100.33 0)
 			(hide yes)
@@
 			)
 		)
-		(property "Datasheet" ""
+		(property "Datasheet" "https://search.murata.co.jp/Ceramy/image/img/A01X/G101/ENG/GCM1555C1HR50BA16-01A.pdf"
 			(at 167.64 83.82 0)
 			(hide yes)
@@
 			)
 		)
-		(property "Description" "100pF, C0G/NP0, ±5%, 50V, 0402 MLCC"
+		(property "Description" "100 pF ±1% 50V Ceramic Capacitor C0G, NP0 0402 (1005 Metric)"
 			(at 167.64 83.82 0)
 			(hide yes)
@@
 			)
 		)
-		(property "Package" "0402"
+		(property "Package" "0402 (1005 Metric)"
 			(at 167.64 83.82 0)
 			(hide yes)
@@
 			)
 		)
-		(property "MPN" "GRM1555C1H101JA01D"
+		(property "MPN" "GCM1555C1H101FA16D"
 			(at 167.64 83.82 0)
 			(hide yes)
@@
 			)
 		)
-		(property "Manufacturer" "Murata"
-			(at 167.64 83.82 0)
-			(hide yes)
-			(show_name no)
-			(do_not_autoplace no)
-			(effects
-				(font
-					(size 1.27 1.27)
-				)
-			)
-		)
-		(property "Suggested Part" "Murata GRM1555C1H101JA01D"
+		(property "Manufacturer" "Murata Electronics"
 			(at 167.64 83.82 0)
 			(hide yes)
@@
 		)
 		(property "Notes" ""
+			(at 167.64 83.82 90)
+			(hide yes)
+			(show_name no)
+			(do_not_autoplace no)
+			(effects
+				(font
+					(size 1.27 1.27)
+				)
+			)
+		)
+		(property "Mount_Type" ""
 			(at 167.64 83.82 90)
 			(hide yes)
@@
 			)
 		)
-		(property "Suggested Part" "Coilcraft 0603CS-68NXJLU"
-			(at 153.67 93.98 0)
-			(hide yes)
-			(show_name no)
-			(do_not_autoplace no)
-			(effects
-				(font
-					(size 1.27 1.27)
-				)
-			)
-		)
 		(property "Purpose" "RF choke/matching inductor in the 1090MHz LNA stage."
 			(at 153.67 93.98 0)
@@
 			(at 153.67 93.98 0)
 			(hide yes)
+			(show_name no)
+			(do_not_autoplace no)
+			(effects
+				(font
+					(size 1.27 1.27)
+				)
+			)
+		)
+		(property "Mount_Type" ""
+			(at 153.67 93.98 0)
+			(hide yes)
