File: planewatcher/kicad/bi_colour_led.kicad_sch (KiCad schematic)
At the start: 3 parts

Commit message: Add persistent PCBWay BOM fields to KiCad schematic
Parts:
- D5: MPN (none) -> APHB1608SGEC; Manufacturer (none) -> Kingbright; Package (none) -> 1608 dual LED
- R3: MPN (none) -> RC0402FR-072K21L; Manufacturer (none) -> Yageo; Package (none) -> 0402
- R4: MPN (none) -> RC0402FR-077K68L; Manufacturer (none) -> Yageo; Package (none) -> 0402
Changed lines of the file:
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@@
+			)
+		)
+		(property "Package" "0402"
+			(at 137.16 62.23 0)
+			(hide yes)
+			(show_name no)
+			(do_not_autoplace no)
+			(effects
+				(font
+					(size 1.27 1.27)
+				)
+			)
+		)
+		(property "MPN" "RC0402FR-077K68L"
+			(at 137.16 62.23 0)
+			(hide yes)
+			(show_name no)
+			(do_not_autoplace no)
+			(effects
+				(font
+					(size 1.27 1.27)
+				)
+			)
+		)
+		(property "Manufacturer" "Yageo"
+			(at 137.16 62.23 0)
+			(hide yes)
+			(show_name no)
+			(do_not_autoplace no)
+			(effects
+				(font
+					(size 1.27 1.27)
+				)
 			)
 		)
@@
 		)
 		(property "Description" "Dual LED, cathodes on pins 2 and 4"
+			(at 172.72 68.58 0)
+			(hide yes)
+			(show_name no)
+			(do_not_autoplace no)
+			(effects
+				(font
+					(size 1.27 1.27)
+				)
+			)
+		)
+		(property "Package" "1608 dual LED"
+			(at 172.72 68.58 0)
+			(hide yes)
+			(show_name no)
+			(do_not_autoplace no)
+			(effects
+				(font
+					(size 1.27 1.27)
+				)
+			)
+		)
+		(property "MPN" "APHB1608SGEC"
+			(at 172.72 68.58 0)
+			(hide yes)
+			(show_name no)
+			(do_not_autoplace no)
+			(effects
+				(font
+					(size 1.27 1.27)
+				)
+			)
+		)
+		(property "Manufacturer" "Kingbright"
 			(at 172.72 68.58 0)
 			(hide yes)
@@
 			(at 148.59 62.23 0)
 			(hide yes)
+			(show_name no)
+			(do_not_autoplace no)
+			(effects
+				(font
+					(size 1.27 1.27)
+				)
+			)
+		)
+		(property "Package" "0402"
+			(at 148.59 62.23 0)
+			(hide yes)
+			(show_name no)
+			(do_not_autoplace no)
+			(effects
+				(font
+					(size 1.27 1.27)
+				)
+			)
+		)
+		(property "MPN" "RC0402FR-072K21L"
+			(at 148.59 62.23 0)
+			(hide yes)
+			(show_name no)
+			(do_not_autoplace no)
+			(effects
+				(font
+					(size 1.27 1.27)
+				)
+			)
+		)
+		(property "Manufacturer" "Yageo"
+			(at 148.59 62.23 0)
+			(hide yes)

Commit message: added lcsc_ids to all parts
Parts:
- D5: lcsc_id (none) -> C7077285
- R3: lcsc_id (none) -> C138019
- R4: lcsc_id (none) -> C155695
Changed lines of the file:
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@@
+			)
+		)
+		(property "lcsc_id" "C155695"
+			(at 137.16 62.23 0)
+			(hide yes)
+			(show_name no)
+			(do_not_autoplace no)
+			(effects
+				(font
+					(size 1.27 1.27)
+				)
 			)
 		)
@@
 		)
 		(property "Manufacturer" "Kingbright"
+			(at 172.72 68.58 0)
+			(hide yes)
+			(show_name no)
+			(do_not_autoplace no)
+			(effects
+				(font
+					(size 1.27 1.27)
+				)
+			)
+		)
+		(property "lcsc_id" "C7077285"
 			(at 172.72 68.58 0)
 			(hide yes)
@@
 			(at 148.59 62.23 0)
 			(hide yes)
+			(show_name no)
+			(do_not_autoplace no)
+			(effects
+				(font
+					(size 1.27 1.27)
+				)
+			)
+		)
+		(property "lcsc_id" "C138019"
+			(at 148.59 62.23 0)
+			(hide yes)
