File: planewatcher/kicad/GPS_Module.kicad_sch (KiCad schematic)
At the start: 9 parts, among them U1 LEA-M8T

Commit message: added lcsc_ids to all parts
Parts:
- C59: MPN GRM188Z71A106MA73J -> GRM188Z71A106MA73D; lcsc_id (none) -> C237435
- C60: lcsc_id (none) -> C161163
- C74: lcsc_id (none) -> C85735
- D4: lcsc_id (none) -> C133346
- R20: lcsc_id (none) -> C4240446
- R21, R23, R24: lcsc_id (none) -> C2935238
Changed lines of the file:
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@@
 			)
 		)
-		(property "MPN" "GRM188Z71A106MA73J"
+		(property "MPN" "GRM188Z71A106MA73D"
 			(at 107.95 55.88 0)
 			(hide yes)
@@
 		(property "Notes" ""
 			(at 107.95 55.88 90)
+			(hide yes)
+			(show_name no)
+			(do_not_autoplace no)
+			(effects
+				(font
+					(size 1.27 1.27)
+				)
+			)
+		)
+		(property "lcsc_id" "C237435"
+			(at 107.95 55.88 0)
 			(hide yes)
 			(show_name no)
@@
 			)
 		)
+		(property "lcsc_id" "C4240446"
+			(at 163.83 59.69 90)
+			(hide yes)
+			(show_name no)
+			(do_not_autoplace no)
+			(effects
+				(font
+					(size 1.27 1.27)
+				)
+			)
+		)
 		(pin "1"
 		)
@@
 			)
 		)
+		(property "lcsc_id" "C85735"
+			(at 179.07 59.69 0)
+			(hide yes)
+			(show_name no)
+			(do_not_autoplace no)
+			(effects
+				(font
+					(size 1.27 1.27)
+				)
+			)
+		)
 		(pin "2"
 		)
@@
 			)
 		)
+		(property "lcsc_id" "C2935238"
+			(at 184.15 127 90)
+			(hide yes)
+			(show_name no)
+			(do_not_autoplace no)
+			(effects
+				(font
+					(size 1.27 1.27)
+				)
+			)
+		)
 		(pin "1"
 		)
@@
 			)
 		)
+		(property "lcsc_id" "C2935238"
+			(at 107.95 81.28 90)
+			(hide yes)
+			(show_name no)
+			(do_not_autoplace no)
+			(effects
+				(font
+					(size 1.27 1.27)
+				)
+			)
+		)
 		(pin "1"
 		)
@@
 			)
 		)
+		(property "lcsc_id" "C133346"
+			(at 184.15 101.6 0)
+			(hide yes)
+			(show_name no)
+			(do_not_autoplace no)
+			(effects
+				(font
+					(size 1.27 1.27)
+				)
+			)
+		)
 		(pin "1"
 		)
@@
 			)
 		)
+		(property "lcsc_id" "C161163"
+			(at 121.92 55.88 0)
+			(hide yes)
+			(show_name no)
+			(do_not_autoplace no)
+			(effects
+				(font
+					(size 1.27 1.27)
+				)
+			)
+		)
 		(pin "1"
 		)
@@
 			(at 107.95 96.52 90)
 			(hide yes)
+			(show_name no)
+			(do_not_autoplace no)
+			(effects
+				(font
+					(size 1.27 1.27)
+				)
+			)
+		)
+		(property "lcsc_id" "C2935238"
+			(at 107.95 96.52 90)
+			(hide yes)

Commit message: change discontinued parts
Parts:
- R21, R23, R24: lcsc_id C2935238 -> C138002
Changed lines of the file:
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@@
 			)
 		)
-		(property "lcsc_id" "C2935238"
+		(property "lcsc_id" "C138002"
 			(at 184.15 127 90)
 			(hide yes)
@@
 			)
 		)
-		(property "lcsc_id" "C2935238"
+		(property "lcsc_id" "C138002"
 			(at 107.95 81.28 90)
 			(hide yes)
@@
 			)
 		)
-		(property "lcsc_id" "C2935238"
+		(property "lcsc_id" "C138002"
 			(at 107.95 96.52 90)
 			(hide yes)

Commit message: update BoM to available parts from LCSC
Parts:
- C74: MPN GRM155R71C103KA01D -> CL05B103KB5NNNC; Manufacturer Murata Electronics -> Samsung Electro-Mechanics; lcsc_id C85735 -> C15195
Changed lines of the file:
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@@
 			)
 		)
-		(property "MPN" "GRM155R71C103KA01D"
+		(property "MPN" "CL05B103KB5NNNC"
 			(at 179.07 59.69 0)
 			(hide yes)
@@
 			)
 		)
-		(property "Manufacturer" "Murata Electronics"
+		(property "Manufacturer" "Samsung Electro-Mechanics"
 			(at 179.07 59.69 0)
 			(hide yes)
@@
 			)
 		)
-		(property "lcsc_id" "C85735"
+		(property "lcsc_id" "C15195"
 			(at 179.07 59.69 0)
 			(hide yes)
