File: planewatcher/kicad/GPS_Module.kicad_sch (KiCad schematic)
At the start: 19 parts, among them J1 1PPS_OUT, U1 LEA-M8T, U4 TC4427

Commit message: Change LCSC column name, add fabrication toolkit options
Parts:
- C59: LCSC (none) -> C237435; lcsc_id C237435 -> (none)
- C60, C62: LCSC (none) -> C161163; lcsc_id C161163 -> (none)
- C63: LCSC (none) -> C913474; lcsc_id C913474 -> (none)
- C74: LCSC (none) -> C15195; lcsc_id C15195 -> (none)
- D4, D5: LCSC (none) -> C133346; lcsc_id C133346 -> (none)
- J1: LCSC (none) -> C88374; lcsc_id C88374 -> (none)
- L10: LCSC (none) -> C3716677; lcsc_id C3716677 -> (none)
- LED6: value PINK LED -> XINGLIGHT XL-1608UPC-06; LCSC (none) -> C2977076; lcsc_id C2977076 -> (none)
- R20: LCSC (none) -> C4240446; lcsc_id C4240446 -> (none)
- R21, R23, R24: LCSC (none) -> C138002; lcsc_id C138002 -> (none)
- R32: LCSC (none) -> C4202009; lcsc_id C4202009 -> (none)
- R33: LCSC (none) -> C77379; lcsc_id C77379 -> (none)
- R47: LCSC (none) -> C481918; lcsc_id C481918 -> (none)
- U1: LCSC (none) -> C2763452; lcsc_id C2763452 -> (none); now not fitted
- U4: LCSC (none) -> C628550; lcsc_id C628550 -> (none)
Changed lines of the file:
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@@
 			(justify left bottom)
 		)
-		(property "Netclass" "RF_50Ω"
+		(property "Net Class" "RF_50Ω"
 			(at 150.4315 71.12 0)
 			(show_name no)
@@
 			(justify left bottom)
 		)
-		(property "Netclass" "RF_50Ω"
+		(property "Net Class" "RF_50Ω"
 			(at 226.6315 90.17 0)
 			(show_name no)
@@
 			)
 		)
-		(property "lcsc_id" "C237435"
+		(property "LCSC" "C237435"
 			(at 49.53 30.48 0)
 			(hide yes)
@@
 			)
 		)
-		(property "lcsc_id" "C4240446"
+		(property "LCSC" "C4240446"
 			(at 124.46 53.34 90)
 			(hide yes)
@@
 			)
 		)
-		(property "lcsc_id" "C4202009"
+		(property "LCSC" "C4202009"
 			(at 207.01 120.65 90)
 			(hide yes)
@@
 			)
 		)
-		(property "lcsc_id" "C3716677"
+		(property "LCSC" "C3716677"
 			(at 34.29 26.67 0)
 			(hide yes)
@@
 			)
 		)
-		(property "lcsc_id" "C161163"
+		(property "LCSC" "C161163"
 			(at 167.64 87.63 0)
 			(hide yes)
@@
 			)
 		)
-		(property "lcsc_id" "C15195"
+		(property "LCSC" "C15195"
 			(at 139.7 53.34 0)
 			(hide yes)
@@
 			)
 		)
-		(property "lcsc_id" "C88374"
+		(property "LCSC" "C88374"
 			(at 236.22 92.71 0)
 			(hide yes)
@@
 			)
 		)
-		(property "lcsc_id" "C628550"
+		(property "LCSC" "C628550"
 			(at 154.94 113.03 0)
 			(hide yes)
@@
 			)
 		)
-		(property "lcsc_id" "C138002"
+		(property "LCSC" "C138002"
 			(at 154.94 148.59 90)
 			(hide yes)
@@
 			)
 		)
-		(property "lcsc_id" "C138002"
+		(property "LCSC" "C138002"
 			(at 38.1 74.93 90)
 			(hide yes)
@@
 			)
 		)
-		(property "lcsc_id" "C481918"
+		(property "LCSC" "C481918"
 			(at 138.43 156.21 0)
 			(hide yes)
@@
 			)
 		)
-		(property "lcsc_id" "C913474"
+		(property "LCSC" "C913474"
 			(at 184.15 87.63 0)
 			(hide yes)
@@
 			)
 		)
-		(property "lcsc_id" "C77379"
+		(property "LCSC" "C77379"
 			(at 208.28 92.71 90)
 			(hide yes)
@@
 			)
 		)
-		(property "lcsc_id" "C133346"
+		(property "LCSC" "C133346"
 			(at 116.84 80.01 0)
 			(hide yes)
@@
 			)
 		)
-		(property "lcsc_id" "C161163"
+		(property "LCSC" "C161163"
 			(at 63.5 30.48 0)
 			(hide yes)
@@
 		(on_board yes)
 		(in_pos_files yes)
-		(dnp no)
+		(dnp yes)
 		(fields_autoplaced yes)
 		(property "Reference" "U1"
@@
 			)
 		)
-		(property "lcsc_id" "C2763452"
+		(property "LCSC" "C2763452"
 			(at 78.74 88.9 0)
 			(hide yes)
@@
 			)
 		)
-		(property "lcsc_id" "C138002"
+		(property "LCSC" "C138002"
 			(at 38.1 90.17 90)
 			(hide yes)
@@
 			)
 		)
-		(property "lcsc_id" "C133346"
+		(property "LCSC" "C133346"
 			(at 214.63 99.06 0)
 			(hide yes)
@@
 			)
 		)
-		(property "Value" "PINK LED"
+		(property "Value" "XINGLIGHT XL-1608UPC-06"
 			(at 192.0875 116.84 0)
 			(show_name no)
@@
 			)
 		)
-		(property "lcsc_id" "C2977076"
+		(property "LCSC" "C2977076"
 			(at 190.5 120.65 0)
 			(hide yes)

Commit message: Adjust component grouping
Parts:
- C60, C62: value 100nF -> 0.1µF
Changed lines of the file:
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@@
 			)
 		)
-		(property "Value" "100nF"
+		(property "Value" "0.1µF"
 			(at 161.798 89.154 0)
 			(show_name no)
@@
 			)
 		)
-		(property "Value" "100nF"
+		(property "Value" "0.1µF"
 			(at 57.658 32.004 0)
 			(show_name no)
