File: planewatcher/kicad/RF_Input.kicad_sch (KiCad schematic)
At the start: 12 parts, among them U2 AP22653AW6-7

Commit message: Add bias-tee power switch & connect GPS TP2
Parts:
- R34: value 20kΩ -> 75kΩ
Other:
- note added: "Sets ~350 mA normal current-limit threshold"
- note removed: "20kΩ sets Ishort to 350mA"
Changed lines of the file:
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@@
 		)
 	)
-	(text "20kΩ sets Ishort to 350mA"
+	(text "Sets ~350 mA normal current-limit threshold"
 		(exclude_from_sim no)
-		(at 109.728 117.602 0)
+		(at 96.52 116.84 0)
 		(effects
 			(font
 				(size 1.27 1.27)
 			)
+			(justify left)
 		)
 	)
@@
 			(width 0)
 			(type default)
-		)
-	)
-	(label "VIN"
-		(at 36.83 93.98 0)
-		(effects
-			(font
-				(size 1.27 1.27)
-			)
-			(justify left bottom)
 		)
 	)
@@
 			)
 		)
-		(property "Value" "20kΩ"
+		(property "Value" "75kΩ"
 			(at 96.52 114.2999 0)
 			(show_name no)

Commit message: Update PCB from schematic & bump version to proto 1.3
Parts:
- LED7: renamed from D1; footprint (none) -> LED_SMD:LED_0603_1608Metric
- LED8: renamed from D5; footprint (none) -> LED_SMD:LED_0603_1608Metric
- R35, R36, R46: footprint (none) -> Resistor_SMD:R_0402_1005Metric
Changed lines of the file:
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@@
 	(title_block
 		(title "Plane Watcher")
-		(date "2026-05-18")
-		(rev "prototype 1.2")
+		(date "2026-06-18")
+		(rev "prototype 1.3")
 		(company "plane.watch")
 		(comment 1 "No warranty; see LICENSE.")
@@
 			)
 		)
-		(property "Footprint" ""
+		(property "Footprint" "Resistor_SMD:R_0402_1005Metric"
 			(at 51.562 142.24 90)
 			(hide yes)
@@
 			)
 		)
-		(property "Footprint" ""
+		(property "Footprint" "Resistor_SMD:R_0402_1005Metric"
 			(at 60.452 138.43 90)
 			(hide yes)
@@
 		(dnp no)
 		(fields_autoplaced yes)
-		(property "Reference" "D5"
+		(property "Reference" "LED8"
 			(at 55.88 131.7624 90)
 			(show_name no)
@@
 			)
 		)
-		(property "Footprint" ""
+		(property "Footprint" "LED_SMD:LED_0603_1608Metric"
 			(at 53.34 134.62 0)
 			(hide yes)
@@
 			(project "planewatcher"
 				(path "/7a4a4324-e8b8-4d06-b75a-28095d4e9f10/688449b3-e085-4d3d-9010-5bd7bcac8461"
-					(reference "D5")
+					(reference "LED8")
 					(unit 1)
 				)
@@
 			)
 		)
-		(property "Footprint" ""
+		(property "Footprint" "Resistor_SMD:R_0402_1005Metric"
 			(at 35.052 116.84 90)
 			(hide yes)
@@
 		(dnp no)
 		(fields_autoplaced yes)
-		(property "Reference" "D1"
+		(property "Reference" "LED7"
 			(at 40.64 124.7774 90)
 			(show_name no)
@@
 			)
 		)
-		(property "Footprint" ""
+		(property "Footprint" "LED_SMD:LED_0603_1608Metric"
 			(at 36.83 124.46 0)
 			(hide yes)
@@
 			(project "planewatcher"
 				(path "/7a4a4324-e8b8-4d06-b75a-28095d4e9f10/688449b3-e085-4d3d-9010-5bd7bcac8461"
-					(reference "D1")
+					(reference "LED7")
 					(unit 1)
 				)

Commit message: Add optional PPS output
Parts:
- added R49: 100kΩ, Resistor_SMD:R_0402_1005Metric, symbol Device:R
- C4: MPN (none) -> GCM155R71A104KA55D; Manufacturer (none) -> Murata Electronics; Package (none) -> 0402 (1005 Metric); Purpose (none) -> Local input bypass capacitor for U2. Provides a low-impedan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; lcsc_id (none) -> C161163
- C5: MPN (none) -> GCM155R71A104KA55D; Manufacturer (none) -> Murata Electronics; Package (none) -> 0402 (1005 Metric); Purpose (none) -> High-frequency output bypass capacitor for the switched bia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; lcsc_id (none) -> C161163
- C6: MPN (none) -> GRM188Z71A106MA73D; Manufacturer (none) -> Murata Electronics; Package (none) -> 0603 (1608 Metric); Purpose (none) -> Bulk output capacitor for the switched bias supply. Support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; lcsc_id (none) -> C237435
- D3: Purpose Provides low-capacitance ESD protection to chassis/board gr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 -> Low-capacitance RF ESD protection from RF centre conductor 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
- L12: Purpose RF choke/shunt inductor; allow bias-tee -> Bias tee RF choke / DC feed inductor. Passes DC bias from U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
- LED7: MPN (none) -> XL-1608PGC-06; Manufacturer (none) -> XINGLIGHT; Purpose (none) -> Bias tee enabled indicator.; lcsc_id (none) -> C7371905
- LED8: MPN (none) -> XL-1608SURC-06; Manufacturer (none) -> XINGLIGHT; Purpose (none) -> Bias tee fault (overcurrent) indicator LED.; lcsc_id (none) -> C965799
- R34: MPN (none) -> CRCW040275K0FKED; Manufacturer (none) -> VISHAY; Package (none) -> 0402 (1005 Metric); Purpose (none) -> Current-limit programming resistor. Sets the normal current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; lcsc_id (none) -> C482234
- R35: MPN (none) -> RC0402FR-071KL; Manufacturer (none) -> YAGEO; Package (none) -> 0402 (1005 Metric); Purpose (none) -> Current-limit resistor for bias tee enable LED.; lcsc_id (none) -> C106235
- R36: MPN (none) -> ERA-2AEB103X; Manufacturer (none) -> Panasonic Industry; Package (none) -> 0402 (1005 Metric); Purpose (none) -> Pull-up resistor for the open-drain FAULT output to LOGIC_V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; lcsc_id (none) -> C191915
- R46: MPN (none) -> RC0402FR-071KL; Manufacturer (none) -> YAGEO; Package (none) -> 0402 (1005 Metric); Purpose (none) -> Current-limit resistor for bias tee fault LED.; lcsc_id (none) -> C106235
- U2: MPN (none) -> AP22653AW6-7; Manufacturer (none) -> DIODES; Package (none) -> SOT-26; Purpose (none) -> Active-high, current-limited high-side power switch for the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; lcsc_id (none) -> C1511768
Connections:
- net BIAS-TEE_EN: now also R49.1
- net GND: now also R49.2
Other:
- note added: "Sets: ILIMIT typ ≈ 319 mA ILIMIT min ≈ 279 mA ILIMIT max ≈ 362 mA"
- note removed: "Sets ~350 mA normal current-limit threshold"
- moved on the sheet: C4, C5, C6, D3, L12, LED7, LED8, R34, R35, R36, R46, U2

Commit message: Tidy up
Parts:
- C6: footprint Capacitor_SMD:C_0402_1005Metric -> Capacitor_SMD:C_0603_1608Metric
- LED7, LED8: Package (none) -> 0603
Changed lines of the file:
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@@
+			)
+		)
+		(property "Package" "0603"
+			(at 102.87 118.11 90)
+			(hide yes)
+			(show_name no)
+			(do_not_autoplace no)
+			(effects
+				(font
+					(size 1.27 1.27)
+				)
 			)
 		)
@@
 			)
 		)
-		(property "Footprint" "Capacitor_SMD:C_0402_1005Metric"
+		(property "Footprint" "Capacitor_SMD:C_0603_1608Metric"
 			(at 169.2148 77.47 0)
 			(hide yes)
@@
 			(at 73.66 111.76 90)
 			(hide yes)
+			(show_name no)
+			(do_not_autoplace no)
+			(effects
+				(font
+					(size 1.27 1.27)
+				)
+			)
+		)
+		(property "Package" "0603"
+			(at 73.66 111.76 90)
+			(hide yes)
