File: planewatcher/kicad/planewatcher.kicad_sch (KiCad schematic)
At the start: 14 parts, among them J2 RF_IN, J3 BMI-S-209-F, J4 FPGA BANK 33, J5 FPGA BANK 35 V1.2/V1.3, J6 GPS _IN

Commit message: Update PCB from schematic & bump version to proto 1.3
Changed lines of the file:
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@@
 	(title_block
 		(title "Plane Watcher")
-		(date "2026-05-18")
-		(rev "prototype 1.2")
+		(date "2026-06-18")
+		(rev "prototype 1.3")
 		(company "plane.watch")
 		(comment 1 "No warranty; see LICENSE.")
@@
 	)
 	(no_connect
-		(at 83.82 148.59)
-	)
-	(no_connect
 		(at 83.82 163.83)
 	)
@@
 	)
 	(no_connect
+		(at 83.82 168.91)
+	)
+	(no_connect
 		(at 83.82 151.13)
 	)
@@
 	)
 	(no_connect
-		(at 127 166.37)
+		(at 127 143.51)
 	)
 	(no_connect
-		(at 83.82 153.67)
+		(at 127 166.37)
 	)
 	(no_connect
-		(at 127 184.15)
+		(at 83.82 153.67)
 	)
 	(no_connect
@@
 	)
 	(no_connect
-		(at 83.82 184.15)
+		(at 127 168.91)
 	)
 	(no_connect
@@
 		)
 	)
+	(label "FPGA_C19"
+		(at 261.62 46.99 180)
+		(effects
+			(font
+				(size 1.27 1.27)
+			)
+			(justify right bottom)
+		)
+	)
 	(label "FPGA_V15"
 		(at 66.04 151.13 180)
@@
 		)
 	)
+	(label "FPGA_H19"
+		(at 26.67 116.84 90)
+		(effects
+			(font
+				(size 1.27 1.27)
+			)
+			(justify left bottom)
+		)
+	)
 	(label "FPGA_V13"
 		(at 270.51 78.74 180)
@@
 		)
 	)
-	(label "FPGA_G15"
-		(at 261.62 46.99 180)
-		(effects
-			(font
-				(size 1.27 1.27)
-			)
-			(justify right bottom)
-		)
-	)
 	(label "FPGA_E15"
 		(at 83.82 151.13 0)
@@
 		)
 	)
-	(label "FPGA_C22"
-		(at 66.04 97.79 180)
-		(effects
-			(font
-				(size 1.27 1.27)
-			)
-			(justify right bottom)
-		)
-	)
 	(label "FPGA_B21"
 		(at 83.82 166.37 0)
@@
 		)
 	)
+	(label "FPGA_H20"
+		(at 66.04 97.79 180)
+		(effects
+			(font
+				(size 1.27 1.27)
+			)
+			(justify right bottom)
+		)
+	)
 	(label "FPGA_B17"
 		(at 127 163.83 180)
@@
 		(effects
 			(font
-				(size 1.27 1.27)
-			)
-			(justify left bottom)
-		)
-	)
-	(label "FPGA_D22"
-		(at 26.67 116.84 90)
-		(effects
-			(font

Commit message: Swap the SMA connectors for U.FL
Parts:
- J2, J6: footprint Connector_Coaxial:SMA_Amphenol_132289_EdgeMount -> Connector_Coaxial:U.FL_Hirose_U.FL-R-SMT-1_Vertical; MPN 132289 -> (none); Manufacturer Amphenol RF -> (none); Package SMA edge-mount -> (none); lcsc_id C3172723 -> (none); now fitted
Changed lines of the file:
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@@
 	(title_block
 		(title "Plane Watcher")
-		(date "2026-06-18")
+		(date "2026-06-19")
 		(rev "prototype 1.3")
 		(company "plane.watch")
@@
 		(on_board yes)
 		(in_pos_files yes)
-		(dnp yes)
+		(dnp no)
 		(property "Reference" "J2"
 			(at 22.1096 78.74 0)
@@
 			)
 		)
-		(property "Footprint" "Connector_Coaxial:SMA_Amphenol_132289_EdgeMount"
+		(property "Footprint" "Connector_Coaxial:U.FL_Hirose_U.FL-R-SMT-1_Vertical"
 			(at 21.59 85.09 0)
 			(hide yes)
@@
 			)
 		)
-		(property "Description" "Right-angle edge-mount SMA jack, 50Ω RF connector"
+		(property "Description" "Hirose U.FL-R-SMT-1, 50Ω RF connector"
 			(at 21.59 85.09 0)
 			(hide yes)
@@
 			)
 		)
-		(property "Package" "SMA edge-mount"
+		(property "Package" ""
 			(at 21.59 85.09 0)
 			(hide yes)
@@
 			)
 		)
-		(property "MPN" "132289"
+		(property "MPN" ""
 			(at 21.59 85.09 0)
 			(hide yes)
@@
 			)
 		)
-		(property "Manufacturer" "Amphenol RF"
+		(property "Manufacturer" ""
 			(at 21.59 85.09 0)
 			(hide yes)
@@
 			)
 		)
-		(property "lcsc_id" "C3172723"
+		(property "lcsc_id" ""
 			(at 21.59 85.09 0)
 			(hide yes)
@@
 		(on_board yes)
 		(in_pos_files yes)
-		(dnp yes)
+		(dnp no)
 		(property "Reference" "J6"
 			(at 217.6896 21.59 0)
@@
 			)
 		)
-		(property "Footprint" "Connector_Coaxial:SMA_Amphenol_132289_EdgeMount"
+		(property "Footprint" "Connector_Coaxial:U.FL_Hirose_U.FL-R-SMT-1_Vertical"
 			(at 217.17 27.94 0)
 			(hide yes)
@@
 			)
 		)
-		(property "Description" "Right-angle edge-mount SMA jack, 50Ω RF connector"
+		(property "Description" "Hirose U.FL-R-SMT-1, 50Ω RF connector"
 			(at 217.17 27.94 0)
 			(hide yes)
@@
 			)
 		)
-		(property "Package" "SMA edge-mount"
+		(property "Package" ""
 			(at 217.17 27.94 0)
 			(hide yes)
@@
 			)
 		)
-		(property "MPN" "132289"
+		(property "MPN" ""
 			(at 217.17 27.94 0)
 			(hide yes)
@@
 			)
 		)
-		(property "Manufacturer" "Amphenol RF"
+		(property "Manufacturer" ""
 			(at 217.17 27.94 0)
 			(hide yes)
@@
 			)
 		)
-		(property "lcsc_id" "C3172723"
+		(property "lcsc_id" ""
 			(at 217.17 27.94 0)
 			(hide yes)

Commit message: Add optional PPS output
Parts:
- J2, J6: MPN (none) -> U.FL-R-SMT-1; Manufacturer (none) -> HRS; Package (none) -> U.FL-R-SMT-1; lcsc_id (none) -> C88374
Changed lines of the file:
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@@
 			)
 		)
-		(property "Datasheet" ""
-			(at 21.59 85.09 0)
-			(hide yes)
-			(show_name no)
-			(do_not_autoplace no)
-			(effects
-				(font
-					(size 1.27 1.27)
-				)
-			)
-		)
-		(property "Description" "Hirose U.FL-R-SMT-1, 50Ω RF connector"
-			(at 21.59 85.09 0)
-			(hide yes)
-			(show_name no)
-			(do_not_autoplace no)
-			(effects
-				(font
-					(size 1.27 1.27)
-				)
-			)
-		)
-		(property "Package" ""
-			(at 21.59 85.09 0)
-			(hide yes)
-			(show_name no)
-			(do_not_autoplace no)
-			(effects
-				(font
-					(size 1.27 1.27)
-				)
-			)
-		)
-		(property "MPN" ""
-			(at 21.59 85.09 0)
-			(hide yes)
-			(show_name no)
-			(do_not_autoplace no)
-			(effects
-				(font
-					(size 1.27 1.27)
-				)
-			)
-		)
-		(property "Manufacturer" ""
+		(property "Datasheet" "https://www.lcsc.com/datasheet/C88374.pdf"
+			(at 21.59 85.09 0)
+			(hide yes)
+			(show_name no)
+			(do_not_autoplace no)
+			(effects
+				(font
+					(size 1.27 1.27)
+				)
+			)
+		)
+		(property "Description" "CONN RCPT IPEX 50Ω SMD"
+			(at 21.59 85.09 0)
+			(hide yes)
+			(show_name no)
+			(do_not_autoplace no)
+			(effects
+				(font
+					(size 1.27 1.27)
+				)
+			)
+		)
+		(property "Package" "U.FL-R-SMT-1"
+			(at 21.59 85.09 0)
+			(hide yes)
+			(show_name no)
+			(do_not_autoplace no)
+			(effects
+				(font
+					(size 1.27 1.27)
+				)
+			)
+		)
+		(property "MPN" "U.FL-R-SMT-1"
+			(at 21.59 85.09 0)
+			(hide yes)
+			(show_name no)
+			(do_not_autoplace no)
+			(effects
+				(font
+					(size 1.27 1.27)
+				)
+			)
+		)
+		(property "Manufacturer" "HRS"
 			(at 21.59 85.09 0)
 			(hide yes)
@@
 			)
 		)
-		(property "lcsc_id" ""
+		(property "lcsc_id" "C88374"
 			(at 21.59 85.09 0)
 			(hide yes)
@@
 			)
 		)
-		(property "Datasheet" ""
-			(at 217.17 27.94 0)
-			(hide yes)
-			(show_name no)
-			(do_not_autoplace no)
-			(effects
-				(font
-					(size 1.27 1.27)
-				)
-			)
-		)
-		(property "Description" "Hirose U.FL-R-SMT-1, 50Ω RF connector"
-			(at 217.17 27.94 0)
-			(hide yes)
-			(show_name no)
-			(do_not_autoplace no)
-			(effects
-				(font
-					(size 1.27 1.27)
-				)
-			)
-		)
-		(property "Package" ""
-			(at 217.17 27.94 0)
-			(hide yes)
-			(show_name no)
-			(do_not_autoplace no)
-			(effects
-				(font
-					(size 1.27 1.27)
-				)
-			)
-		)
-		(property "MPN" ""
-			(at 217.17 27.94 0)
-			(hide yes)
-			(show_name no)
-			(do_not_autoplace no)
-			(effects
-				(font
-					(size 1.27 1.27)
-				)
-			)
-		)
-		(property "Manufacturer" ""
+		(property "Datasheet" "https://www.lcsc.com/datasheet/C88374.pdf"
+			(at 217.17 27.94 0)
+			(hide yes)
+			(show_name no)
+			(do_not_autoplace no)
+			(effects
+				(font
+					(size 1.27 1.27)
+				)
+			)
+		)
+		(property "Description" "CONN RCPT IPEX 50Ω SMD"
+			(at 217.17 27.94 0)
+			(hide yes)
+			(show_name no)
+			(do_not_autoplace no)
+			(effects
+				(font
+					(size 1.27 1.27)
+				)
+			)
+		)
+		(property "Package" "U.FL-R-SMT-1"
+			(at 217.17 27.94 0)
+			(hide yes)
+			(show_name no)
+			(do_not_autoplace no)
+			(effects
+				(font
+					(size 1.27 1.27)
+				)
+			)
+		)
+		(property "MPN" "U.FL-R-SMT-1"
+			(at 217.17 27.94 0)
+			(hide yes)
+			(show_name no)
+			(do_not_autoplace no)
+			(effects
+				(font
+					(size 1.27 1.27)
+				)
+			)
+		)
+		(property "Manufacturer" "HRS"
 			(at 217.17 27.94 0)
 			(hide yes)
@@
 			)
 		)
-		(property "lcsc_id" ""
-			(at 217.17 27.94 0)
-			(hide yes)
+		(property "lcsc_id" "C88374"
+			(at 217.17 27.94 0)
+			(hide yes)

Commit message: Update PCB to include PPS output
Other:
- sheet GPS Module ports: added 3V3, 4V5; removed VCC
Changed lines of the file:
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@@
 	)
 	(junction
+		(at 62.23 22.86)
+		(diameter 0)
+		(color 0 0 0 0)
+	)
+	(junction
 		(at 120.65 34.29)
 		(diameter 0)
@@
 	(wire
 		(pts
+			(xy 62.23 22.86) (xy 66.04 22.86)
+		)
+		(stroke
+			(width 0)
+			(type default)
+		)
+	)
+	(wire
+		(pts
 			(xy 193.04 85.09) (xy 199.39 85.09)
 		)
@@
 	(wire
 		(pts
+			(xy 208.28 43.18) (xy 226.06 43.18)
+		)
+		(stroke
+			(width 0)
+			(type default)
+		)
+	)
+	(wire
+		(pts
 			(xy 250.19 36.83) (xy 261.62 36.83)
 		)
@@
 	(wire
 		(pts
-			(xy 57.15 22.86) (xy 66.04 22.86)
+			(xy 57.15 22.86) (xy 62.23 22.86)
 		)
 		(stroke
@@
 		)
 	)
+	(label "4V5"
+		(at 208.28 43.18 0)
+		(effects
+			(font
+				(size 1.27 1.27)
+			)
+			(justify left bottom)
+		)
+	)
 	(label "FPGA_Y18"
 		(at 270.51 86.36 180)
@@
 	)
 	(symbol
+		(lib_id "power:+3.3VADC")
+		(at 62.23 22.86 0)
+		(unit 1)
+		(body_style 1)
+		(exclude_from_sim no)
+		(in_bom yes)
+		(on_board yes)
+		(in_pos_files yes)
+		(dnp no)
+		(property "Reference" "#PWR043"
+			(at 66.04 24.13 0)
+			(hide yes)
+			(show_name no)
+			(do_not_autoplace no)
+			(effects
+				(font
+					(size 1.27 1.27)
+				)
+			)
+		)
+		(property "Value" "4V5"
+			(at 62.23 18.796 0)
+			(show_name no)
+			(do_not_autoplace no)
+			(effects
+				(font
+					(size 1.27 1.27)
+				)
+			)
+		)
+		(property "Footprint" ""
+			(at 62.23 22.86 0)
+			(hide yes)
+			(show_name no)
+			(do_not_autoplace no)
+			(effects
+				(font
+					(size 1.27 1.27)
+				)
+			)
+		)
+		(property "Datasheet" ""
+			(at 62.23 22.86 0)
+			(hide yes)
+			(show_name no)
+			(do_not_autoplace no)
+			(effects
+				(font
+					(size 1.27 1.27)
+				)
+			)
+		)
+		(property "Description" "Power symbol creates a global label with name \"+3.3VADC\""
+			(at 62.23 22.86 0)
+			(hide yes)
+			(show_name no)
+			(do_not_autoplace no)
+			(effects
+				(font
+					(size 1.27 1.27)
+				)
+			)
+		)
+		(pin "1"
+		)
+		(instances
+			(project "planewatcher"
+				(path "/7a4a4324-e8b8-4d06-b75a-28095d4e9f10"
+					(reference "#PWR043")
+					(unit 1)
+				)
+			)
+		)
+	)
+	(symbol
 		(lib_id "power:GND")
 		(at 73.66 173.99 0)
@@
 			)
 		)
-		(pin "VCC" input
-			(at 226.06 39.37 180)
-			(effects
-				(font
-					(size 1.27 1.27)
-				)
-				(justify left)
-			)
-		)
 		(pin "RF_IN" input
 			(at 238.76 33.02 90)
@@
 			)
 		)
+		(pin "3V3" input
+			(at 226.06 39.37 180)
+			(effects
+				(font
+					(size 1.27 1.27)
+				)
+				(justify left)
+			)
+		)
+		(pin "4V5" input
+			(at 226.06 43.18 180)
+			(effects
+				(font
+					(size 1.27 1.27)
+				)
+				(justify left)
+			)
+		)

Commit message: Implement log detector output buffering & buffered low-pass filter for noise offset
- Implement low-pass filter to output noise floor with no pulses
- Feed noise floor into ADC driver -IN to improve range/sensitivity
- Buffer low pass filter output
- Buffer log detector output with spare op amp in OPA2320 package
- Tidy schematic & vias
Other:
- sheet ADC ports: added none; removed VREF
- sheet ADC_Driver ports: added none; removed ADC_OFFSET
Changed lines of the file:
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@@
 	(wire
 		(pts
-			(xy 227.33 90.17) (xy 233.68 90.17)
-		)
-		(stroke
-			(width 0)
-			(type default)
-		)
-	)
-	(wire
-		(pts
 			(xy 22.86 191.77) (xy 38.1 191.77)
 		)
@@
 	(sheet
 		(at 199.39 77.47)
-		(size 27.94 15.24)
+		(size 27.94 10.16)
 		(exclude_from_sim no)
 		(in_bom yes)
@@
 		)
 		(property "Sheetfile" "ADC_Driver.kicad_sch"
-			(at 199.39 93.2946 0)
+			(at 199.39 88.2146 0)
 			(show_name no)
 			(do_not_autoplace no)
@@
 			)
 		)
-		(pin "ADC_OFFSET" input
-			(at 227.33 90.17 0)
-			(effects
-				(font
-					(size 1.27 1.27)
-				)
-				(justify right)
-			)
-		)
 		(instances
 			(project "planewatcher"
@@
 			)
 		)
-		(pin "VREF" output
-			(at 233.68 90.17 180)
-			(effects
-				(font
-					(size 1.27 1.27)
-				)
-				(justify left)
-			)
-		)

Commit message: Replace TADJ prototype trimmer with voltage divider
Voltage divider sets the ADL5513 TADJ pin to approximately 0.85 V for 1090 MHz operation
Parts:
- J3: value BMI-S-209-F -> BMI-S-209-F + C; MPN BMI-S-209-F -> BMI-S-209-F + BMI-S-209-C
Changed lines of the file:
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@@
 			)
 		)
-		(property "Value" "BMI-S-209-F"
+		(property "Value" "BMI-S-209-F + C"
 			(at 195.58 101.5999 0)
 			(show_name no)
@@
 			)
 		)
-		(property "MPN" "BMI-S-209-F"
+		(property "MPN" "BMI-S-209-F + BMI-S-209-C"
 			(at 179.07 100.33 0)
 			(hide yes)
