File: planewatcher/kicad/fpga_headers_bank_35.kicad_sch (KiCad schematic)
At the start: 1 part, among them J5 FPGA BANK 35 V1.2/V1.3

Commit message: Populate Z13 with 68nH
After initial testing of the prototype 1.3, Z13 was populated with 68nH which improved RF performance significantly.
Other:
- company: (none) -> plane.watch
- title: (none) -> Plane Watcher
Changed lines of the file:
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@@
 	(paper "A4")
 	(title_block
+		(title "Plane Watcher")
+		(date "2026-09-25")
+		(rev "1.4")
+		(company "plane.watch")
+		(comment 1 "No warranty; see LICENSE.")
 		(comment 2 "Source: https://github.com/plane-watch/hardware.")
 		(comment 3 "Licensed under CERN-OHL-S-2.0.")
@@
 					(reference "J5")
 					(unit 1)
-				)
-			)
+					(variant
+						(name "revision_1.4")
+					)
+				)
+			)
