File: planewatcher/kicad/ADC.kicad_sch (KiCad schematic)
At the start: 24 parts, among them U11 AD9203

Commit message: Change LCSC column name, add fabrication toolkit options
Parts:
- C49, C52, C55, C58: LCSC (none) -> C237435; lcsc_id C237435 -> (none)
- C50, C51, C53, C54, C56, C57: LCSC (none) -> C161163; lcsc_id C161163 -> (none)
- C68, C73, C77: LCSC (none) -> C126493; lcsc_id C126493 -> (none)
- C69, C75, C76: LCSC (none) -> C2941926; lcsc_id C2941926 -> (none)
- L6, L9: LCSC (none) -> C3716677; lcsc_id C3716677 -> (none)
- R4, R5: LCSC (none) -> C242160; lcsc_id C242160 -> (none)
- RN2, RN3, RN4: LCSC (none) -> C1734385; lcsc_id C1734385 -> (none)
- U11: value AD9203 -> AD9203ARUZ; LCSC (none) -> C653239; lcsc_id C653239 -> (none)
Changed lines of the file:
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@@
 			)
 		)
-		(property "lcsc_id" "C237435"
+		(property "LCSC" "C237435"
 			(at 264.16 85.09 0)
 			(hide yes)
@@
 			)
 		)
-		(property "lcsc_id" "C126493"
+		(property "LCSC" "C126493"
 			(at 86.36 25.4 0)
 			(hide yes)
@@
 			)
 		)
-		(property "lcsc_id" "C161163"
+		(property "LCSC" "C161163"
 			(at 250.19 85.09 0)
 			(hide yes)
@@
 			)
 		)
-		(property "lcsc_id" "C126493"
+		(property "LCSC" "C126493"
 			(at 203.2 25.4 0)
 			(hide yes)
@@
 			)
 		)
-		(property "lcsc_id" "C1734385"
+		(property "LCSC" "C1734385"
 			(at 110.49 69.85 0)
 			(hide yes)
@@
 			)
 		)
-		(property "lcsc_id" "C3716677"
+		(property "LCSC" "C3716677"
 			(at 44.45 21.59 0)
 			(hide yes)
@@
 			)
 		)
-		(property "lcsc_id" "C237435"
+		(property "LCSC" "C237435"
 			(at 233.68 62.23 0)
 			(hide yes)
@@
 			)
 		)
-		(property "lcsc_id" "C161163"
+		(property "LCSC" "C161163"
 			(at 219.71 62.23 0)
 			(hide yes)
@@
 			)
 		)
-		(property "lcsc_id" "C161163"
+		(property "LCSC" "C161163"
 			(at 72.39 25.4 0)
 			(hide yes)
@@
 			)
 		)
-		(property "lcsc_id" "C161163"
+		(property "LCSC" "C161163"
 			(at 217.17 25.4 0)
 			(hide yes)
@@
 			)
 		)
-		(property "lcsc_id" "C237435"
+		(property "LCSC" "C237435"
 			(at 231.14 25.4 0)
 			(hide yes)
@@
 			)
 		)
-		(property "lcsc_id" "C2941926"
+		(property "LCSC" "C2941926"
 			(at 189.23 25.4 0)
 			(hide yes)
@@
 			)
 		)
-		(property "lcsc_id" "C3716677"
+		(property "LCSC" "C3716677"
 			(at 251.46 21.59 0)
 			(hide yes)
@@
 			)
 		)
-		(property "Value" "AD9203"
+		(property "Value" "AD9203ARUZ"
 			(at 148.59 34.29 0)
 			(show_name no)
@@
 			)
 		)
-		(property "lcsc_id" "C653239"
+		(property "LCSC" "C653239"
 			(at 148.59 34.29 0)
 			(hide yes)
@@
 			)
 		)
-		(property "lcsc_id" "C2941926"
+		(property "LCSC" "C2941926"
 			(at 222.25 85.09 0)
 			(hide yes)
@@
 			)
 		)
-		(property "lcsc_id" "C237435"
+		(property "LCSC" "C237435"
 			(at 58.42 25.4 0)
 			(hide yes)
@@
 			)
 		)
-		(property "lcsc_id" "C126493"
+		(property "LCSC" "C126493"
 			(at 236.22 85.09 0)
 			(hide yes)
@@
 			)
 		)
-		(property "lcsc_id" "C242160"
+		(property "LCSC" "C242160"
 			(at 186.69 81.28 90)
 			(hide yes)
@@
 			)
 		)
-		(property "lcsc_id" "C161163"
+		(property "LCSC" "C161163"
 			(at 250.19 66.04 0)
 			(hide yes)
@@
 			)
 		)
-		(property "lcsc_id" "C242160"
+		(property "LCSC" "C242160"
 			(at 180.34 88.9 0)
 			(hide yes)
@@
 			)
 		)
-		(property "lcsc_id" "C1734385"
+		(property "LCSC" "C1734385"
 			(at 110.49 54.61 0)
 			(hide yes)
@@
 			)
 		)
-		(property "lcsc_id" "C1734385"
+		(property "LCSC" "C1734385"
 			(at 110.49 82.55 0)
 			(hide yes)
@@
 			)
 		)
-		(property "lcsc_id" "C2941926"
+		(property "LCSC" "C2941926"
 			(at 100.33 25.4 0)
 			(hide yes)
@@
 			)
 		)
-		(property "lcsc_id" "C161163"
+		(property "LCSC" "C161163"
 			(at 250.19 58.42 0)
 			(hide yes)

Commit message: Adjust component grouping
Parts:
- C50, C51, C53, C54, C56, C57: value 100nF -> 0.1µF
Changed lines of the file:
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@@
 			)
 		)
-		(property "Value" "100nF"
+		(property "Value" "0.1µF"
 			(at 254 86.3599 0)
 			(show_name no)
@@
 			)
 		)
-		(property "Value" "100nF"
+		(property "Value" "0.1µF"
 			(at 223.52 63.4999 0)
 			(show_name no)
@@
 			)
 		)
-		(property "Value" "100nF"
+		(property "Value" "0.1µF"
 			(at 76.2 26.6699 0)
 			(show_name no)
@@
 			)
 		)
-		(property "Value" "100nF"
+		(property "Value" "0.1µF"
 			(at 220.98 26.6699 0)
 			(show_name no)
@@
 			)
 		)
-		(property "Value" "100nF"
+		(property "Value" "0.1µF"
 			(at 250.19 73.66 90)
 			(show_name no)
@@
 			)
 		)
-		(property "Value" "100nF"
+		(property "Value" "0.1µF"
 			(at 250.19 53.34 90)
 			(show_name no)

Commit message: Add comments & markup to schematic
Changed lines of the file:
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@@
 		(exclude_from_sim no)
 		(at 213.36 78.74 0)
-		(size 60.96 30.48)
+		(size 60.96 20.32)
 		(margins 0.9525 0.9525 0.9525 0.9525)
 		(stroke
@@
 		(exclude_from_sim no)
 		(at 213.36 44.45 0)
-		(size 69.85 31.75)
+		(size 60.96 31.75)
 		(margins 0.9525 0.9525 0.9525 0.9525)
 		(stroke
