File: planewatcher/kicad/LNA_Stage_2.kicad_sch (KiCad schematic)
At the start: 14 parts, among them U7 TQP3M9036

Commit message: Update symbols to Kicad 10.0.5
Parts:
- Z14: renamed from Z13; value 68nH -> TBD; LCSC C3221883 -> (none); MPN 0402DC-68NXJRW -> (none); Manufacturer Coilcraft -> (none); now not fitted; now left out of the parts list
- renumbered C28 to C34, C29 to C35, C30 to C36, C31 to C37, C32 to C38, C33 to C39, L7 to L8, Z8 to R9, U7 to U8, Z15 to Z16, Z17 to Z19, Z12 to Z20, Z18 to Z21
Changed lines of the file:
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@@
 		(dnp yes)
 		(fields_autoplaced yes)
-		(property "Reference" "Z17"
+		(property "Reference" "Z19"
 			(at 194.31 109.2199 0)
 			(show_name no)
@@
 		(dnp no)
 		(fields_autoplaced yes)
-		(property "Reference" "#PWR059"
+		(property "Reference" "#PWR066"
 			(at 173.99 52.07 0)
 			(hide yes)
@@
 		(dnp no)
 		(fields_autoplaced yes)
-		(property "Reference" "C28"
+		(property "Reference" "C34"
 			(at 167.64 38.1 90)
 			(show_name no)
@@
 		(dnp no)
 		(fields_autoplaced yes)
-		(property "Reference" "#PWR065"
+		(property "Reference" "#PWR072"
 			(at 132.08 139.7 0)
 			(hide yes)
@@
 		(dnp no)
 		(fields_autoplaced yes)
-		(property "Reference" "#PWR064"
+		(property "Reference" "#PWR071"
 			(at 153.67 132.08 0)
 			(hide yes)
@@
 		(dnp no)
 		(fields_autoplaced yes)
-		(property "Reference" "#PWR0117"
+		(property "Reference" "#PWR0119"
 			(at 204.47 120.65 0)
 			(hide yes)
@@
 		(dnp no)
 		(fields_autoplaced yes)
-		(property "Reference" "#PWR061"
+		(property "Reference" "#PWR068"
 			(at 173.99 77.47 0)
 			(hide yes)
@@
 		(dnp no)
 		(fields_autoplaced yes)
-		(property "Reference" "C32"
+		(property "Reference" "C38"
 			(at 110.49 96.52 90)
 			(show_name no)
@@
 		(dnp no)
 		(fields_autoplaced yes)
-		(property "Reference" "#PWR0116"
+		(property "Reference" "#PWR0118"
 			(at 191.77 120.65 0)
 			(hide yes)
@@
 		(dnp no)
 		(fields_autoplaced yes)
-		(property "Reference" "C33"
+		(property "Reference" "C39"
 			(at 167.64 96.52 90)
 			(show_name no)
@@
 		(dnp no)
 		(fields_autoplaced yes)
-		(property "Reference" "Z12"
+		(property "Reference" "Z20"
 			(at 198.12 97.79 90)
 			(show_name no)
@@
 		(dnp no)
 		(fields_autoplaced yes)
-		(property "Reference" "Z8"
+		(property "Reference" "R9"
 			(at 83.82 97.79 90)
 			(show_name no)
@@
 		(dnp no)
 		(fields_autoplaced yes)
-		(property "Reference" "C29"
+		(property "Reference" "C35"
 			(at 167.64 50.8 90)
 			(show_name no)
@@
 		(body_style 1)
 		(exclude_from_sim no)
-		(in_bom yes)
+		(in_bom no)
 		(on_board yes)
 		(in_pos_files yes)
-		(dnp no)
+		(dnp yes)
 		(fields_autoplaced yes)
-		(property "Reference" "Z13"
+		(property "Reference" "Z14"
 			(at 80.01 109.2199 0)
 			(show_name no)
@@
 			)
 		)
-		(property "Value" "68nH"
+		(property "Value" "TBD"
 			(at 80.01 111.7599 0)
 			(show_name no)
@@
 			)
 		)
-		(property "Description" "First shunt element in pi pad, populated after initial testing of proto 1.3"
+		(property "Description" "First shunt element in pi pad"
 			(at 77.47 110.49 0)
 			(hide yes)
@@
 			)
 		)
-		(property "LCSC" "C3221883"
+		(property "LCSC" ""
 			(at 77.47 110.49 0)
 			(hide yes)
@@
 			)
 		)
-		(property "MPN" "0402DC-68NXJRW"
+		(property "MPN" ""
 			(at 77.47 110.49 0)
 			(hide yes)
@@
 			)
 		)
-		(property "Manufacturer" "Coilcraft"
+		(property "Manufacturer" ""
 			(at 77.47 110.49 0)
 			(hide yes)
@@
 		(dnp no)
 		(fields_autoplaced yes)
-		(property "Reference" "C30"
+		(property "Reference" "C36"
 			(at 167.64 63.5 90)
 			(show_name no)
@@
 		(dnp yes)
 		(fields_autoplaced yes)
-		(property "Reference" "Z18"
+		(property "Reference" "Z21"
 			(at 207.01 109.2199 0)
 			(show_name no)
@@
 		(dnp no)
 		(fields_autoplaced yes)
-		(property "Reference" "U7"
+		(property "Reference" "U8"
 			(at 139.065 110.49 0)
 			(show_name no)
@@
 		(dnp no)
 		(fields_autoplaced yes)
-		(property "Reference" "#PWR060"
+		(property "Reference" "#PWR067"
 			(at 173.99 64.77 0)
 			(hide yes)
@@
 		(dnp yes)
 		(fields_autoplaced yes)
-		(property "Reference" "Z15"
+		(property "Reference" "Z16"
 			(at 92.71 109.2199 0)
 			(show_name no)
@@
 		(dnp no)
 		(fields_autoplaced yes)
-		(property "Reference" "C31"
+		(property "Reference" "C37"
 			(at 167.64 76.2 90)
 			(show_name no)
@@
 		(dnp no)
 		(fields_autoplaced yes)
-		(property "Reference" "#PWR062"
+		(property "Reference" "#PWR069"
 			(at 173.99 90.17 0)
 			(hide yes)
@@
 		(dnp no)
 		(fields_autoplaced yes)
-		(property "Reference" "#PWR0112"
+		(property "Reference" "#PWR0113"
 			(at 90.17 120.65 0)
 			(hide yes)
@@
 		(dnp no)
 		(fields_autoplaced yes)
-		(property "Reference" "L7"
+		(property "Reference" "L8"
 			(at 154.94 92.7099 0)
 			(show_name no)
@@
 		(dnp no)
 		(fields_autoplaced yes)
-		(property "Reference" "#PWR052"
+		(property "Reference" "#PWR053"
 			(at 77.47 120.65 0)
 			(hide yes)
@@
 		(dnp no)
 		(fields_autoplaced yes)
-		(property "Reference" "#PWR063"
+		(property "Reference" "#PWR070"
 			(at 124.46 132.08 0)
 			(hide yes)

Commit message: Add comments & markup to schematic
Changed lines of the file:
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@@
 		)
 	)
-	(text_box "Pi pad for RF matching"
+	(text_box "Pi pad for RF matching\n\nDNP pads & 0ΩR allow for future population of L/C/R components to improve impedance (Z) matching."
 		(exclude_from_sim no)
 		(at 69.85 95.25 0)
-		(size 27.94 30.48)
+		(size 27.94 41.91)
 		(margins 0.9525 0.9525 0.9525 0.9525)
 		(stroke
@@
 		)
 	)
-	(text_box "Pi pad for RF matching"
-		(exclude_from_sim no)
-		(at 184.15 95.25 0)
-		(size 27.94 30.48)
+	(text_box "RF block,\nDC pass"
+		(exclude_from_sim no)
+		(at 142.24 87.63 0)
+		(size 19.05 12.7)
 		(margins 0.9525 0.9525 0.9525 0.9525)
 		(stroke
@@
 				(size 1.27 1.27)
 			)
+			(justify left)
+		)
+	)
+	(text_box "Pi pad for RF matching\n\nDNP pads & 0ΩR allow for future population of L/C/R components to improve impedance (Z) matching."
+		(exclude_from_sim no)
+		(at 184.15 95.25 0)
+		(size 27.94 41.91)
+		(margins 0.9525 0.9525 0.9525 0.9525)
+		(stroke
+			(width 0)
+			(type solid)
+		)
+		(fill
+			(type none)
+		)
+		(effects
+			(font
+				(size 1.27 1.27)
+			)
 			(justify left bottom)
 		)
 	)
+	(text_box "DC block,\nRF pass"
+		(exclude_from_sim no)
+		(at 105.41 95.25 0)
+		(size 11.43 20.32)
+		(margins 0.9525 0.9525 0.9525 0.9525)
+		(stroke
+			(width 0)
+			(type solid)
+		)
+		(fill
+			(type none)
+		)
+		(effects
+			(font
+				(size 1.27 1.27)
+			)
+			(justify bottom)
+		)
+	)
+	(text_box "DC block,\nRF pass"
+		(exclude_from_sim no)
+		(at 162.56 95.25 0)
+		(size 11.43 20.32)
+		(margins 0.9525 0.9525 0.9525 0.9525)
+		(stroke
+			(width 0)
+			(type solid)
+		)
+		(fill
+			(type none)
+		)
+		(effects
+			(font
+				(size 1.27 1.27)
+			)
+			(justify bottom)
+		)
+	)
+	(text_box "Shutdown tied to \nGND for always-on."
+		(exclude_from_sim no)
+		(at 153.67 120.65 0)
+		(size 26.67 13.97)
+		(margins 0.9525 0.9525 0.9525 0.9525)
+		(stroke
+			(width 0)
+			(type solid)
+		)
+		(fill
+			(type none)
+		)
+		(effects
+			(font
+				(size 1.27 1.27)
+			)
+			(justify right)
+		)
+	)
 	(text_box "RF_IN and RF_OUT are 50Ω controlled-impedance RF traces.\nKeep short. No stubs. Reference solid GND plane."
 		(exclude_from_sim no)
-		(at 104.14 76.2 0)
+		(at 57.15 80.01 0)
 		(size 34.29 11.43)
 		(margins 0.9525 0.9525 0.9525 0.9525)
@@
 		)
 	)
+	(text_box "Supply decoupling\n& bypassing."
+		(exclude_from_sim no)
+		(at 162.56 35.56 0)
+		(size 33.02 55.88)
+		(margins 0.9525 0.9525 0.9525 0.9525)
+		(stroke
+			(width 0)
+			(type solid)
+		)
+		(fill
+			(type none)
+		)
+		(effects
+			(font
+				(size 1.27 1.27)
+			)
+			(justify right)
+		)
+	)
 	(junction
 		(at 139.7 133.35)
@@
 		(pts
 			(xy 153.67 71.12) (xy 153.67 83.82)
+		)
+		(stroke
+			(width 0)
+			(type default)
+		)
+	)
+	(wire
+		(pts
+			(xy 157.48 125.73) (xy 153.67 125.73)
 		)
 		(stroke
@@
 	(symbol
 		(lib_id "power:GND")
-		(at 153.67 125.73 0)
+		(at 157.48 125.73 0)
 		(unit 1)
 		(body_style 1)
@@
 		(fields_autoplaced yes)
 		(property "Reference" "#PWR071"
-			(at 153.67 132.08 0)
+			(at 157.48 132.08 0)
 			(hide yes)
 			(show_name no)
@@
 		)
 		(property "Value" "GND"
-			(at 153.67 130.81 0)
+			(at 157.48 130.81 0)
 			(show_name no)
 			(do_not_autoplace no)
@@
 		)
 		(property "Footprint" ""
-			(at 153.67 125.73 0)
+			(at 157.48 125.73 0)
 			(hide yes)
 			(show_name no)
@@
 		)
 		(property "Datasheet" ""
-			(at 153.67 125.73 0)
+			(at 157.48 125.73 0)
 			(hide yes)
 			(show_name no)
@@
 		)
 		(property "Description" "Power symbol creates a global label with name \"GND\" , ground"
-			(at 153.67 125.73 0)
-			(hide yes)
-			(show_name no)
+			(at 157.48 125.73 0)
+			(hide yes)
+			(show_name no)
