File: planewatcher/kicad/PowerStage_LDO.kicad_sch (KiCad schematic)
At the start: 13 parts, among them U6 LT3045/LT3045-1

Commit message: Change LCSC column name, add fabrication toolkit options
Parts:
- C19, C21: LCSC (none) -> C51205; lcsc_id C51205 -> (none)
- C2, C22: LCSC (none) -> C161163; lcsc_id C161163 -> (none)
- C26: LCSC (none) -> C913474; lcsc_id C913474 -> (none)
- C27: LCSC (none) -> C87996; lcsc_id C87996 -> (none)
- C3: LCSC (none) -> C126493; lcsc_id C126493 -> (none)
- L5: LCSC (none) -> C3716677; lcsc_id C3716677 -> (none)
- R18: LCSC (none) -> C191915; lcsc_id C191915 -> (none)
- R19: LCSC (none) -> C2088785; lcsc_id C2088785 -> (none)
- R22: LCSC (none) -> C860335; lcsc_id C860335 -> (none)
- TP1: now not fitted
- U6: LCSC (none) -> C666587; lcsc_id C666587 -> (none)
Changed lines of the file:
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@@
 			)
 		)
-		(property "lcsc_id" "C3716677"
+		(property "LCSC" "C3716677"
 			(at 83.82 83.82 0)
 			(hide yes)
@@
 			)
 		)
-		(property "lcsc_id" "C51205"
+		(property "LCSC" "C51205"
 			(at 121.92 87.63 0)
 			(hide yes)
@@
 			)
 		)
-		(property "lcsc_id" "C87996"
+		(property "LCSC" "C87996"
 			(at 194.31 99.06 0)
 			(hide yes)
@@
 			)
 		)
-		(property "lcsc_id" "C126493"
+		(property "LCSC" "C126493"
 			(at 222.25 99.06 0)
 			(hide yes)
@@
 			)
 		)
-		(property "lcsc_id" "C860335"
+		(property "LCSC" "C860335"
 			(at 149.86 120.65 0)
 			(hide yes)
@@
 			)
 		)
-		(property "lcsc_id" "C191915"
+		(property "LCSC" "C191915"
 			(at 139.7 67.31 0)
 			(hide yes)
@@
 			)
 		)
-		(property "lcsc_id" "C161163"
+		(property "LCSC" "C161163"
 			(at 209.55 99.06 0)
 			(hide yes)
@@
 		(on_board yes)
 		(in_pos_files yes)
-		(dnp no)
+		(dnp yes)
 		(fields_autoplaced yes)
 		(property "Reference" "TP1"
@@
 			)
 		)
-		(property "lcsc_id" "C666587"
+		(property "LCSC" "C666587"
 			(at 166.37 76.2 0)
 			(hide yes)
@@
 			)
 		)
-		(property "lcsc_id" "C51205"
+		(property "LCSC" "C51205"
 			(at 57.15 87.63 0)
 			(hide yes)
@@
 			)
 		)
-		(property "lcsc_id" "C913474"
+		(property "LCSC" "C913474"
 			(at 137.16 120.65 0)
 			(hide yes)
@@
 			)
 		)
-		(property "lcsc_id" "C161163"
+		(property "LCSC" "C161163"
 			(at 92.71 87.63 0)
 			(hide yes)
@@
 			)
 		)
-		(property "lcsc_id" "C2088785"
+		(property "LCSC" "C2088785"
 			(at 149.86 67.31 0)
 			(hide yes)

Commit message: Adjust component grouping
Parts:
- C2, C22: value 100nF -> 0.1µF
Changed lines of the file:
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@@
 			)
 		)
-		(property "Value" "100nF"
+		(property "Value" "0.1µF"
 			(at 213.36 100.3299 0)
 			(show_name no)
@@
 			)
 		)
-		(property "Value" "100nF"
+		(property "Value" "0.1µF"
 			(at 96.52 88.8999 0)
 			(show_name no)

Commit message: fix invalid footprint name
Parts:
- U6: footprint planewatcher:U_LT3045IMSE-1#PBF -> planewatcher:U_LT3045IMSE-1_PBF
Changed lines of the file:
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@@
 			)
 		)
-		(property "Footprint" "planewatcher:U_LT3045IMSE-1#PBF"
+		(property "Footprint" "planewatcher:U_LT3045IMSE-1_PBF"
 			(at 166.37 76.2 0)
 			(hide yes)

Commit message: Add comments & markup to schematic
Changed lines of the file:
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@@
 		)
 	)
-	(text_box "${/7a4a4324-e8b8-4d06-b75a-28095d4e9f10/e02d84ed-6468-4290-a59c-50ded41c0aba/d0620f5f-b1cf-4df8-a6ae-ece97448600e:REFERENCE} marked DNP to adhere to USB capacitance limit (although FPGA board waaaaay exceeds the limit anyway..."
+	(text_box "${/7a4a4324-e8b8-4d06-b75a-28095d4e9f10/e02d84ed-6468-4290-a59c-50ded41c0aba/d0620f5f-b1cf-4df8-a6ae-ece97448600e:REFERENCE} marked DNP to adhere to USB capacitance limit (although FPGA board waaaaay exceeds the limit anyway...)"
 		(exclude_from_sim no)
 		(at 43.18 81.28 0)
