File: planewatcher/kicad/RGB_LEDs.kicad_sch (KiCad schematic)
At the start: 7 parts

Commit message: Change LCSC column name, add fabrication toolkit options
Parts:
- LED1, LED2, LED3, LED4, LED5: LCSC (none) -> C5145179; lcsc_id C5145179 -> (none)
- RN5, RN6: LCSC (none) -> C874618; lcsc_id C874618 -> (none)
Changed lines of the file:
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@@
 			)
 		)
-		(property "lcsc_id" "C5145179"
+		(property "LCSC" "C5145179"
 			(at 52.07 130.81 0)
 			(hide yes)
@@
 			)
 		)
-		(property "lcsc_id" "C5145179"
+		(property "LCSC" "C5145179"
 			(at 52.07 80.01 0)
 			(hide yes)
@@
 			)
 		)
-		(property "lcsc_id" "C5145179"
+		(property "LCSC" "C5145179"
 			(at 52.07 105.41 0)
 			(hide yes)
@@
 			)
 		)
-		(property "lcsc_id" "C5145179"
+		(property "LCSC" "C5145179"
 			(at 52.07 29.21 0)
 			(hide yes)
@@
 			)
 		)
-		(property "lcsc_id" "C874618"
+		(property "LCSC" "C874618"
 			(at 115.57 34.29 90)
 			(hide yes)
@@
 			)
 		)
-		(property "lcsc_id" "C874618"
+		(property "LCSC" "C874618"
 			(at 115.57 66.04 90)
 			(hide yes)
@@
 			)
 		)
-		(property "lcsc_id" "C5145179"
+		(property "LCSC" "C5145179"
 			(at 52.07 54.61 0)
 			(hide yes)

Commit message: Add comments & markup to schematic
Other:
- note added: "RELAXEN UND WATSCHEN DER BLINKENLIGHTS :-)"
Changed lines of the file:
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@@
 		(comment 4 "Copyright (C) 2026 plane.watch team and contributors.")
+	)
+	(text "RELAXEN UND WATSCHEN DER BLINKENLIGHTS :-)"
+		(exclude_from_sim no)
+		(at 52.07 144.272 0)
+		(effects
+			(font
+				(size 1.27 1.27)
+			)
+		)
 	)
 	(junction
