File: planewatcher/kicad/eeprom.kicad_sch (KiCad schematic)
At the start: 5 parts, among them U5 24LC16BT-I/OT

Commit message: Update BoM with EEPROM componentry details
Parts:
- R6, R7: MPN (none) -> ERJ2RKF2001X; Manufacturer (none) -> Panasonic Industry; Package (none) -> 0402 (1005 Metric); Purpose (none) -> Pull-up for EEPROM data lines, for 400MHz operation as-per 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; lcsc_id (none) -> C413086
- U5: MPN (none) -> 24LC16BT-I/OT; Manufacturer (none) -> MICROCHIP; Package (none) -> SOT-23-5; Purpose (none) -> EEPROM for board serial & config details.; lcsc_id (none) -> C2061286
Changed lines of the file:
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@@
+			)
+		)
+		(property "MPN" "24LC16BT-I/OT"
+			(at 147.32 87.63 0)
+			(hide yes)
+			(show_name no)
+			(do_not_autoplace no)
+			(effects
+				(font
+					(size 1.27 1.27)
+				)
+			)
+		)
+		(property "Manufacturer" "MICROCHIP"
+			(at 147.32 87.63 0)
+			(hide yes)
+			(show_name no)
+			(do_not_autoplace no)
+			(effects
+				(font
+					(size 1.27 1.27)
+				)
+			)
+		)
+		(property "Package" "SOT-23-5"
+			(at 147.32 87.63 0)
+			(hide yes)
+			(show_name no)
+			(do_not_autoplace no)
+			(effects
+				(font
+					(size 1.27 1.27)
+				)
+			)
+		)
+		(property "Purpose" "EEPROM for board serial & config details."
+			(at 147.32 87.63 0)
+			(hide yes)
+			(show_name no)
+			(do_not_autoplace no)
+			(effects
+				(font
+					(size 1.27 1.27)
+				)
+			)
+		)
+		(property "lcsc_id" "C2061286"
+			(at 147.32 87.63 0)
+			(hide yes)
+			(show_name no)
+			(do_not_autoplace no)
+			(effects
+				(font
+					(size 1.27 1.27)
+				)
 			)
 		)
@@
 			)
 		)
-		(property "Datasheet" ""
+		(property "Datasheet" "https://www.lcsc.com/datasheet/C413086.pdf"
 			(at 172.72 85.09 0)
 			(hide yes)
@@
 			)
 		)
-		(property "Description" "Resistor"
+		(property "Description" "RES 2kΩ ±1% 100mW 0402"
+			(at 172.72 85.09 0)
+			(hide yes)
+			(show_name no)
+			(do_not_autoplace no)
+			(effects
+				(font
+					(size 1.27 1.27)
+				)
+			)
+		)
+		(property "MPN" "ERJ2RKF2001X"
+			(at 172.72 85.09 0)
+			(hide yes)
+			(show_name no)
+			(do_not_autoplace no)
+			(effects
+				(font
+					(size 1.27 1.27)
+				)
+			)
+		)
+		(property "Manufacturer" "Panasonic Industry"
+			(at 172.72 85.09 0)
+			(hide yes)
+			(show_name no)
+			(do_not_autoplace no)
+			(effects
+				(font
+					(size 1.27 1.27)
+				)
+			)
+		)
+		(property "Package" "0402 (1005 Metric)"
+			(at 172.72 85.09 0)
+			(hide yes)
+			(show_name no)
+			(do_not_autoplace no)
+			(effects
+				(font
+					(size 1.27 1.27)
+				)
+			)
+		)
+		(property "Purpose" "Pull-up for EEPROM data lines, for 400MHz operation as-per datasheet."
+			(at 172.72 85.09 0)
+			(hide yes)
+			(show_name no)
+			(do_not_autoplace no)
+			(effects
+				(font
+					(size 1.27 1.27)
+				)
+			)
+		)
+		(property "lcsc_id" "C413086"
 			(at 172.72 85.09 0)
 			(hide yes)
@@
 			)
 		)
-		(property "Datasheet" ""
+		(property "Datasheet" "https://www.lcsc.com/datasheet/C413086.pdf"
 			(at 184.15 85.09 0)
 			(hide yes)
@@
 			)
 		)
-		(property "Description" "Resistor"
+		(property "Description" "RES 2kΩ ±1% 100mW 0402"
 			(at 184.15 85.09 0)
 			(hide yes)
+			(show_name no)
+			(do_not_autoplace no)
+			(effects
+				(font
+					(size 1.27 1.27)
+				)
+			)
+		)
+		(property "MPN" "ERJ2RKF2001X"
+			(at 184.15 85.09 0)
+			(hide yes)
+			(show_name no)
+			(do_not_autoplace no)
+			(effects
+				(font
+					(size 1.27 1.27)
+				)
+			)
+		)
+		(property "Manufacturer" "Panasonic Industry"
+			(at 184.15 85.09 0)
+			(hide yes)
+			(show_name no)
+			(do_not_autoplace no)
+			(effects
+				(font
+					(size 1.27 1.27)
+				)
+			)
+		)
+		(property "Package" "0402 (1005 Metric)"
+			(at 184.15 85.09 0)
+			(hide yes)
+			(show_name no)
+			(do_not_autoplace no)
+			(effects
+				(font
+					(size 1.27 1.27)
+				)
+			)
+		)
+		(property "Purpose" "Pull-up for EEPROM data lines, for 400MHz operation as-per datasheet."
+			(at 184.15 85.09 0)
+			(hide yes)
+			(show_name no)
+			(do_not_autoplace no)
+			(effects
+				(font
+					(size 1.27 1.27)
+				)
+			)
+		)
+		(property "lcsc_id" "C413086"
+			(at 184.15 85.09 0)
+			(hide yes)

Commit message: Add RF pi matching networks + more
- Remove EEPROM write project solder jumper
- Update proto 1.3 documentation
Parts:
- removed JP1: Write Protect, Jumper:SolderJumper-3_P1.3mm_Bridged12_RoundedPad1.0x1.5mm_NumberLabels, symbol Jumper:SolderJumper_3_Bridged12
Connections:
- net GND: now also U5.5 (WP)
Other:
- note removed: "1-2: Normal 2-3: Write Inhibited"
Changed lines of the file:
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@@
 		(comment 4 "Copyright (C) 2026 plane.watch team and contributors.")
-	)
-	(text "1-2: Normal\n2-3: Write Inhibited"
-		(exclude_from_sim no)
-		(at 94.996 108.204 0)
-		(effects
-			(font
-				(size 1.27 1.27)
-			)
-			(justify left)
-		)
-	)
-	(text_box "Write protect solder jumper"
-		(exclude_from_sim no)
-		(at 93.98 92.71 0)
-		(size 39.37 17.78)
-		(margins 0.9525 0.9525 0.9525 0.9525)
-		(stroke
-			(width 0)
-			(type solid)
-		)
-		(fill
-			(type none)
-		)
-		(effects
-			(font
-				(size 1.27 1.27)
-			)
-			(justify left top)
-		)
 	)
 	(text_box "Pull-ups for 400MHz operation"
@@
 	)
 	(junction
-		(at 147.32 86.36)
-		(diameter 0)
-		(color 0 0 0 0)
-	)
-	(junction
 		(at 147.32 76.2)
 		(diameter 0)
@@
 	(wire
 		(pts
-			(xy 147.32 76.2) (xy 147.32 86.36)
-		)
-		(stroke
-			(width 0)
-			(type default)
-		)
-	)
-	(wire
-		(pts
 			(xy 147.32 76.2) (xy 118.11 76.2)
 		)
@@
 	(wire
 		(pts
-			(xy 128.27 95.25) (xy 128.27 86.36)
-		)
-		(stroke
-			(width 0)
-			(type default)
-		)
-	)
-	(wire
-		(pts
 			(xy 156.21 99.06) (xy 184.15 99.06)
 		)
@@
 	(wire
 		(pts
-			(xy 128.27 86.36) (xy 147.32 86.36)
-		)
-		(stroke
-			(width 0)
-			(type default)
-		)
-	)
-	(wire
-		(pts
 			(xy 172.72 76.2) (xy 172.72 81.28)
 		)
@@
 	(wire
 		(pts
-			(xy 135.89 100.33) (xy 135.89 96.52)
+			(xy 135.89 96.52) (xy 135.89 105.41)
 		)
 		(stroke
@@
 	(wire
 		(pts
-			(xy 132.08 100.33) (xy 135.89 100.33)
+			(xy 135.89 105.41) (xy 147.32 105.41)
 		)
 		(stroke
@@
 	(wire
 		(pts
-			(xy 128.27 105.41) (xy 147.32 105.41)
-		)
-		(stroke
-			(width 0)
-			(type default)
-		)
-	)
-	(wire
-		(pts
-			(xy 147.32 86.36) (xy 147.32 88.9)
+			(xy 147.32 76.2) (xy 147.32 88.9)
 		)
 		(stroke
@@
 					(unit 1)
 				)
-			)
-		)
-	)
-	(symbol
-		(lib_id "Jumper:SolderJumper_3_Bridged12")
-		(at 128.27 100.33 90)
-		(unit 1)
-		(body_style 1)
-		(exclude_from_sim no)
-		(in_bom no)
-		(on_board yes)
-		(in_pos_files yes)
-		(dnp no)
-		(fields_autoplaced yes)
-		(property "Reference" "JP1"
-			(at 125.73 99.0599 90)
-			(show_name no)
-			(do_not_autoplace no)
-			(effects
-				(font
-					(size 1.27 1.27)
-				)
-				(justify left)
-			)
-		)
-		(property "Value" "Write Protect"
-			(at 125.73 101.5999 90)
-			(show_name no)
-			(do_not_autoplace no)
-			(effects
-				(font
-					(size 1.27 1.27)
-				)
-				(justify left)
-			)
-		)
-		(property "Footprint" "Jumper:SolderJumper-3_P1.3mm_Bridged12_RoundedPad1.0x1.5mm_NumberLabels"
-			(at 128.27 100.33 0)
-			(hide yes)
-			(show_name no)
-			(do_not_autoplace no)
-			(effects
-				(font
-					(size 1.27 1.27)
-				)
-			)
-		)
-		(property "Datasheet" ""
-			(at 143.51 100.33 0)
-			(hide yes)
-			(show_name no)
-			(do_not_autoplace no)
-			(effects
-				(font
-					(size 1.27 1.27)
-				)
-			)
-		)
-		(property "Description" "3-pole Solder Jumper, pins 1+2 closed/bridged"
-			(at 140.97 100.33 0)
-			(hide yes)
-			(show_name no)
-			(do_not_autoplace no)
-			(effects
-				(font
-					(size 1.27 1.27)
-				)
-			)
-		)
-		(pin "3"
-		)
-		(pin "1"
-		)
-		(pin "2"
-		)
-		(instances
-			(project "planewatcher"
-				(path "/7a4a4324-e8b8-4d06-b75a-28095d4e9f10/51edb038-216c-41f2-9cc3-d6f88328fe89"
-					(reference "JP1")
-					(unit 1)
-				)

Commit message: Change LCSC column name, add fabrication toolkit options
Parts:
- C83: LCSC (none) -> C161163; lcsc_id C161163 -> (none)
- R6, R7: LCSC (none) -> C413086; lcsc_id C413086 -> (none)
- U5: LCSC (none) -> C2061286; lcsc_id C2061286 -> (none)
Changed lines of the file:
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@@
 			)
 		)
-		(property "lcsc_id" "C2061286"
+		(property "LCSC" "C2061286"
 			(at 147.32 87.63 0)
 			(hide yes)
@@
 			)
 		)
-		(property "lcsc_id" "C161163"
+		(property "LCSC" "C161163"
 			(at 118.11 80.01 0)
 			(hide yes)
@@
 			)
 		)
-		(property "lcsc_id" "C413086"
+		(property "LCSC" "C413086"
 			(at 172.72 85.09 0)
 			(hide yes)
@@
 			)
 		)
-		(property "lcsc_id" "C413086"
-			(at 184.15 85.09 0)
-			(hide yes)
+		(property "LCSC" "C413086"
+			(at 184.15 85.09 0)
+			(hide yes)

Commit message: Adjust component grouping
Parts:
- C83: value 100nF -> 0.1µF
Changed lines of the file:
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@@
 			)
 		)
-		(property "Value" "100nF"
+		(property "Value" "0.1µF"
 			(at 112.268 81.534 0)
 			(show_name no)

Commit message: Add comments & markup to schematic
Changed lines of the file:
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@@
+		)
+	)
+	(text_box "Write Protect (WP, pin 5) tied to ground to enable writing."
+		(exclude_from_sim no)
+		(at 114.3 93.98 0)
+		(size 24.13 20.32)
+		(margins 0.9525 0.9525 0.9525 0.9525)
+		(stroke
+			(width 0)
+			(type solid)
+		)
+		(fill
+			(type none)
+		)
+		(effects
+			(font
+				(size 1.27 1.27)
+			)
+			(justify left bottom)
+		)
+	)
+	(text_box "Every prototype 1.3 (and later boards) store the hardware identity in this Microchip 24LC16B EEPROM.\n\nThe EEPROM data is written once at assembly time and read back at boot-time to set board details such as MAC address, serial number, credentials, etc.\n"
+		(exclude_from_sim no)
+		(at 115.57 124.46 0)
+		(size 62.23 15.24)
+		(margins 0.9525 0.9525 0.9525 0.9525)
+		(stroke
+			(width 0)
+			(type solid)
+		)
+		(fill
+			(type none)
+		)
+		(effects
+			(font
+				(size 1.27 1.27)
+			)
+			(justify left top)
 		)
 	)
